Commit message: modified:   README.md 	modified:   cho_controller/cho_controller_franka/include/cho_controller_franka/base_controller.hpp 	modified:   cho_controller/cho_controller_franka/src/base_controller.cpp 	modified:   cho_controller/cho_controller_franka/src/gravity_compensation_controller.cpp 	modified:   cho_controller/cho_controller_franka/src/joint_space_impedance_controller.cpp 	modified:   cho_controller/cho_controller_franka/src/joint_space_qp_controller.cpp 	modified:   cho_controller/cho_controller_franka/src/operational_space_controller.cpp 	modified:   cho_controller/cho_controller_franka/src/task_space_impedance_controller.cpp 	modified:   cho_controller/cho_controller_franka/src/task_space_qp_controller.cpp 	modified:   cho_controller/cho_controller_franka/src/vla_controller.cpp 	modified:   cho_robots_bringup/cho_franka_bringup/config/gazebo/controllers.yaml 	modified:   cho_robots_bringup/cho_franka_bringup/launch/bringup_gazebo_robot.launch.py 	modified:   cho_robots_description/cho_franka_description/robots/common/franka_arm.ros2_control.xacro 	modified:   cho_task_manager/python/plot_pose_log.py

File: cho_robots_description/cho_franka_description/robots/common/franka_arm.ros2_control.xacro (robot description, xacro)
@@ -31,5 +31,5 @@
         </hardware>
       <!-- Joint position, velocity and effort interfaces -->
-      <xacro:macro name="configure_joint" params="joint_name initial_position">
+      <xacro:macro name="configure_joint" params="joint_name initial_position is_gripper:=false">
         <joint name="${joint_name}">
           <!--
@@ -39,5 +39,5 @@
             <command_interface name="position"/>
             <command_interface name="velocity"/>
-          <xacro:if value="${gazebo == 0 or gazebo_effort == 1}">
+          <xacro:if value="${gazebo == 0 or gazebo_effort == 1 or is_gripper == 1}">
             <command_interface name="effort"/>
           </xacro:if>
@@ -59,5 +59,5 @@
       <xacro:configure_joint joint_name="${arm_prefix}${robot_type}_joint7" initial_position="${pi/4}"/>
       <xacro:if value="${gazebo and hand}">
-        <xacro:configure_joint joint_name="${arm_prefix}${robot_type}_finger_joint1" initial_position="0.0" />
+        <xacro:configure_joint joint_name="${arm_prefix}${robot_type}_finger_joint1" initial_position="0.0" is_gripper="true" />
       </xacro:if>
       <xacro:macro name="general_purpose_io" params="prefix command_interface index">
