Commit message: change vla_controller gain

File: cho_robots_description/cho_franka_description/robots/common/franka_robot.xacro (robot description, xacro)
@@ -52,12 +52,11 @@
       <link name="${special_connection}">
         <inertial>
-          <mass value="0.24"/>
-          <origin xyz="0 0 0.019"/>
+          <mass value="0.24"/> <!-- Adjust mass based on your sensor specs -->
+          <origin xyz="0 0 0"/>
           <inertia ixx="0.001" ixy="0.0" ixz="0.0" iyy="0.001" iyz="0.0" izz="0.001"/>
         </inertial>
         <visual>
-          <origin xyz="0 0 0.019" rpy="0 0 0"/>
           <geometry>
-            <cylinder radius="0.035" length="0.038"/>
+            <cylinder radius="0.035" length="0.035"/>
           </geometry>
           <material name="sensor_material">
@@ -67,7 +66,7 @@
       </link>
       <joint name="flange_to_${special_connection}" type="fixed">
-        <parent link="${arm_prefix}${robot_type}_link8"/>
+        <parent link="${arm_prefix}${robot_type}_link8"/> <!-- This is the end-effector flange -->
         <child link="${special_connection}"/>
-        <origin xyz="0 0 0" rpy="0 0 0"/>
+        <origin xyz="0 0 0.0175"/> <!-- Adjust based on sensor position -->
       </joint>
     </xacro:unless>

File: cho_robots_description/cho_franka_description/urdf/fr3_with_ft_sensor/fr3_franka_hand.urdf (robot description, URDF)
Before this commit: robot fr3, 36 links, 35 joints
Joints:
- joint flange_to_ft_sensor: origin xyz=0 0 0 rpy=0 0 0 -> xyz=0 0 0.0175 rpy=0 0 0
- joint fr3_hand_joint: origin xyz=0 0 0.035 rpy=0 0 -0.7853981633974483 -> xyz=0 0 0.0175 rpy=0 0 -0.7853981633974483

Commit message: modified:   cho_controller/cho_controller_franka/include/cho_controller_franka/base_controller.hpp 	modified:   cho_controller/cho_controller_franka/src/base_controller.cpp 	modified:   cho_controller/cho_controller_franka/src/servers/task_space_action_server.cpp 	modified:   cho_robots_bringup/cho_franka_bringup/config/payload.yaml 	modified:   cho_robots_bringup/cho_franka_bringup/launch/bringup_gazebo_robot.launch.py 	deleted:    cho_robots_bringup/cho_franka_bringup/launch/bringup_real_robot.launch copy.py 	modified:   cho_robots_bringup/cho_franka_bringup/launch/bringup_real_robot.launch.py 	modified:   cho_robots_description/cho_franka_description/robots/common/franka_robot.xacro 	modified:   cho_robots_description/cho_franka_description/urdf/fr3_with_ft_sensor/fr3_franka_hand.urdf 	modified:   cho_task_manager/cho_task_manager/tasks/__init__.py 	modified:   cho_task_manager/cho_task_manager/utils/controller_names.py 	modified:   cho_task_manager/cho_task_manager/utils/msg_utils.py

File: cho_robots_description/cho_franka_description/robots/common/franka_robot.xacro (robot description, xacro)
@@ -54,5 +54,5 @@
           <mass value="0.24"/> <!-- Adjust mass based on your sensor specs -->
           <origin xyz="0 0 0"/>
-          <inertia ixx="0.001" ixy="0.0" ixz="0.0" iyy="0.001" iyz="0.0" izz="0.001"/>
+          <inertia ixx="0.000098" ixy="0.0" ixz="0.0" iyy="0.000098" iyz="0.0" izz="0.0001470"/>
         </inertial>
         <visual>

Commit message: modified:   cho_robots_bringup/cho_franka_bringup/launch/bringup_gazebo_robot.launch.py 	modified:   cho_robots_bringup/cho_franka_bringup/launch/bringup_real_robot.launch.py 	modified:   cho_robots_bringup/cho_franka_bringup/launch/bringup_real_robot_backup.launch.py 	modified:   cho_robots_description/cho_franka_description/robots/common/franka_robot.xacro 	modified:   cho_robots_description/cho_franka_description/urdf/fr3_with_ft_sensor/fr3_franka_hand.urdf

File: cho_robots_description/cho_franka_description/robots/common/franka_robot.xacro (robot description, xacro)
@@ -68,5 +68,5 @@
         <parent link="${arm_prefix}${robot_type}_link8"/> <!-- This is the end-effector flange -->
         <child link="${special_connection}"/>
-        <origin xyz="0 0 0.0175"/> <!-- Adjust based on sensor position -->
+        <origin xyz="0 0 0.0175" rpy="${pi} 0 0"/> <!-- Adjust based on sensor position -->
       </joint>
     </xacro:unless>

File: cho_robots_description/cho_franka_description/urdf/fr3_with_ft_sensor/fr3_franka_hand.urdf (robot description, URDF)
Before this commit: robot fr3, 36 links, 35 joints
Joints:
- joint flange_to_ft_sensor: origin xyz=0 0 0.0175 rpy=0 0 0 -> xyz=0 0 0.0175 rpy=3.141592653589793 0 0
- joint fr3_hand_joint: origin xyz=0 0 0.0175 rpy=0 0 -0.7853981633974483 -> xyz=0 0 -0.0175 rpy=3.141592653589793 0 0.7853981633974483

Commit message: modified:   cho_robots_bringup/cho_franka_bringup/launch/bringup_gazebo_robot.launch.py 	modified:   cho_robots_bringup/cho_franka_bringup/launch/bringup_real_robot.launch.py 	modified:   cho_robots_bringup/cho_franka_bringup/launch/bringup_real_robot_backup.launch.py 	modified:   cho_robots_description/cho_franka_description/robots/common/franka_robot.xacro 	modified:   cho_robots_description/cho_franka_description/urdf/fr3_with_ft_sensor/fr3_franka_hand.urdf

File: cho_robots_description/cho_franka_description/robots/common/franka_robot.xacro (robot description, xacro)
@@ -68,5 +68,5 @@
         <parent link="${arm_prefix}${robot_type}_link8"/> <!-- This is the end-effector flange -->
         <child link="${special_connection}"/>
-        <origin xyz="0 0 0.0175" rpy="${pi} 0 0"/> <!-- Adjust based on sensor position -->
+        <origin xyz="0 0 0.0175" rpy="0 0 0"/> <!-- Adjust based on sensor position -->
       </joint>
     </xacro:unless>

File: cho_robots_description/cho_franka_description/urdf/fr3_with_ft_sensor/fr3_franka_hand.urdf (robot description, URDF)
Before this commit: robot fr3, 36 links, 35 joints
Joints:
- joint flange_to_ft_sensor: origin xyz=0 0 0.0175 rpy=3.141592653589793 0 0 -> xyz=0 0 0.0175 rpy=0 0 0
- joint fr3_hand_joint: origin xyz=0 0 -0.0175 rpy=3.141592653589793 0 0.7853981633974483 -> xyz=0 0 0.0175 rpy=0 0 -0.7853981633974483

Commit message: modified:   README.md 	modified:   cho_controller/cho_controller_franka/CMakeLists.txt 	modified:   cho_controller/cho_controller_franka/cho_controller_franka.xml 	modified:   cho_controller/cho_controller_franka/include/cho_controller_franka/base_controller.hpp 	new file:   cho_controller/cho_controller_franka/include/cho_controller_franka/joint_space_position_controller.hpp 	modified:   cho_controller/cho_controller_franka/include/cho_controller_franka/servers/base_action_server.hpp 	modified:   cho_controller/cho_controller_franka/include/cho_controller_franka/servers/joint_space_action_server.hpp 	modified:   cho_controller/cho_controller_franka/include/cho_controller_franka/servers/task_space_action_server.hpp 	modified:   cho_controller/cho_controller_franka/include/cho_controller_franka/task_space_ik_controller.hpp 	modified:   cho_controller/cho_controller_franka/src/base_controller.cpp 	new file:   cho_controller/cho_controller_franka/src/joint_space_position_controller.cpp 	modified:   cho_controller/cho_controller_franka/src/servers/joint_space_action_server.cpp 	modified:   cho_controller/cho_controller_franka/src/servers/task_space_action_server.cpp 	modified:   cho_controller/cho_controller_franka/src/task_space_ik_controller.cpp 	modified:   cho_controller/cho_controller_ur/CMakeLists.txt 	modified:   cho_controller/cho_controller_ur/cho_controller_ur.xml 	renamed:    cho_controller/cho_controller_ur/include/cho_controller_ur/joint_space_controller.hpp -> cho_controller/cho_controller_ur/include/cho_controller_ur/joint_space_position_controller.hpp 	renamed:    cho_controller/cho_controller_ur/src/joint_space_controller.cpp -> cho_controller/cho_controller_ur/src/joint_space_position_controller.cpp 	modified:   cho_controller/cho_controller_ur/src/task_space_ik_controller.cpp 	modified:   cho_robots_bringup/cho_franka_bringup/config/gazebo/controllers.yaml 	modified:   cho_robots_bringup/cho_franka_bringup/config/mujoco/controllers.yaml 	modified:   cho_robots_bringup/cho_franka_bringup/config/real/controllers.yaml 	modified:   cho_robots_bringup/cho_franka_bringup/launch/bringup_gz_robot.launch.py 	modified:   cho_robots_bringup/cho_franka_bringup/launch/bringup_real_robot.launch.py 	modified:   cho_robots_bringup/cho_franka_bringup/utils/launch_utils.py 	modified:   cho_robots_bringup/cho_ur_bringup/config/gz/controllers.yaml 	modified:   cho_robots_bringup/cho_ur_bringup/config/mujoco/controllers.yaml 	modified:   cho_robots_bringup/cho_ur_bringup/config/real/controllers.yaml 	modified:   cho_robots_bringup/cho_ur_bringup/config/real/ur5e.config.yaml 	modified:   cho_robots_bringup/cho_ur_bringup/launch/bringup_gz_robot.launch.py 	modified:   cho_robots_bringup/cho_ur_bringup/launch/bringup_mujoco_robot.launch.py 	modified:   cho_robots_bringup/cho_ur_bringup/launch/bringup_real_robot.launch.py 	new file:   cho_robots_description/cho_franka_description/meshes/accessories/ft_sensor/mounting.stl 	modified:   cho_robots_description/cho_franka_description/robots/common/franka_robot.xacro 	modified:   cho_robots_description/cho_franka_description/urdf/fr3/fr3_franka_hand.urdf 	modified:   cho_robots_description/cho_franka_description/urdf/fr3_with_ft_sensor/fr3_franka_hand.urdf 	new file:   cho_robots_description/cho_franka_description/xml/fr3/actuators_position.xml 	new file:   cho_robots_description/cho_franka_description/xml/fr3/actuators_torque.xml 	modified:   cho_robots_description/cho_franka_description/xml/fr3/fr3.xml 	new file:   cho_robots_description/cho_franka_description/xml/fr3/scene_position.xml 	new file:   cho_robots_description/cho_franka_description/xml/fr3/scene_torque.xml 	new file:   cho_robots_description/cho_franka_description/xml/fr3_with_ft_sensor/actuators_position.xml 	new file:   cho_robots_description/cho_franka_description/xml/fr3_with_ft_sensor/actuators_torque.xml 	new file:   cho_robots_description/cho_franka_description/xml/fr3_with_ft_sensor/assets/mounting.stl 	modified:   cho_robots_description/cho_franka_description/xml/fr3_with_ft_sensor/fr3.xml 	new file:   cho_robots_description/cho_franka_description/xml/fr3_with_ft_sensor/scene_position.xml 	new file:   cho_robots_description/cho_franka_description/xml/fr3_with_ft_sensor/scene_torque.xml

File: cho_robots_description/cho_franka_description/robots/common/franka_robot.xacro (robot description, xacro)
@@ -48,26 +48,72 @@
       connected_to="${connected_to}"
     />
-    <!-- Force-Torque Sensor Link -->
+    <!-- Bota SensONE Force-Torque Sensor -->
     <xacro:unless value="${special_connection == ''}">
-      <link name="${special_connection}">
+      <!-- Mounting part bolted to the arm flange (link8) -->
+      <joint name="robot_mounting_link_to_bota_ft_sensor" type="fixed">
+        <parent link="${arm_prefix}${robot_type}_link8"/>
+        <child link="bota_ft_sensor_mounting"/>
+        <origin rpy="0 0 0" xyz="0 0 0"/>
+      </joint>
+      <link name="bota_ft_sensor_mounting">
         <inertial>
-          <mass value="0.24"/> <!-- Adjust mass based on your sensor specs -->
-          <origin xyz="0 0 0"/>
-          <inertia ixx="0.000098" ixy="0.0" ixz="0.0" iyy="0.000098" iyz="0.0" izz="0.0001470"/>
+          <origin rpy="0 0 0" xyz="-0.00011559 0.00060052 0.010067"/>
+          <mass value="0.15393"/>
+          <inertia ixx="4.907E-05" ixy="3.2541E-08" ixz="-1.0415E-07" iyy="5.5735E-05" iyz="1.3709E-07" izz="9.0228E-05"/>
         </inertial>
         <visual>
+          <origin rpy="0 0 0" xyz="0 0 0"/>
           <geometry>
-            <cylinder radius="0.035" length="0.035"/>
+            <mesh filename="package://cho_franka_description/meshes/accessories/ft_sensor/mounting.stl"/>
           </geometry>
-          <material name="sensor_material">
-            <color rgba="0.1 0.1 0.1 1.0"/>
+          <material name="bota_ft_material">
+            <color rgba="0.6902 0.61176 0.52941 1"/>
           </material>
         </visual>
+        <collision>
+          <origin rpy="0 0 0" xyz="0 0 0.011"/>
+          <geometry><cylinder length="0.028" radius="0.035"/></geometry>
+        </collision>
+        <collision>
+          <origin rpy="1.57 0 0" xyz="0 0.051 0.0115"/>
+          <geometry><cylinder length="0.032" radius="0.0065"/></geometry>
+        </collision>
+        <collision>
+          <origin rpy="0 0 0" xyz="0 0 0.03"/>
+          <geometry><cylinder length="0.01" radius="0.0315"/></geometry>
+        </collision>
       </link>
-      <joint name="flange_to_${special_connection}" type="fixed">
-        <parent link="${arm_prefix}${robot_type}_link8"/> <!-- This is the end-effector flange -->
-        <child link="${special_connection}"/>
-        <origin xyz="0 0 0.0175" rpy="0 0 0"/> <!-- Adjust based on sensor position -->
-      </joint>
+      <!-- Wrench (force/torque measurement) frame, 35 mm above the mounting base -->
+      <joint name="bota_ft_sensor_mounting_to_wrench" type="fixed">
+        <origin rpy="0 0 0" xyz="0 0 0.035"/>
+        <parent link="bota_ft_sensor_mounting"/>
+        <child link="bota_ft_sensor_wrench"/>
+      </joint>
+      <link name="bota_ft_sensor_wrench">
+        <inertial>
+          <origin rpy="0 0 0" xyz="-0.00018335 -3.3341E-07 -0.0070612"/>
+          <mass value="0.08253"/>
+          <inertia ixx="2.2674E-05" ixy="-3.9222E-12" ixz="4.8952E-08" iyy="2.2294E-05" iyz="4.0972E-11" izz="4.0919E-05"/>
+        </inertial>
+      </link>
+      <!-- Internal mechanical reference frames -->
+      <joint name="bota_ft_sensor_mounting_to_mech1" type="fixed">
+        <origin rpy="1.5625 0 -1.5708" xyz="-0.032879 0 0.0105"/>
+        <parent link="bota_ft_sensor_mounting"/>
+        <child link="bota_ft_sensor_mech1"/>
+      </joint>
+      <link name="bota_ft_sensor_mech1"/>
+      <joint name="bota_ft_sensor_mounting_to_mech2" type="fixed">
+        <origin rpy="1.5708 0 0" xyz="0 -0.032879 0.0105"/>
+        <parent link="bota_ft_sensor_mounting"/>
+        <child link="bota_ft_sensor_mech2"/>
+      </joint>
+      <link name="bota_ft_sensor_mech2"/>
+      <joint name="bota_ft_sensor_mounting_to_mech3" type="fixed">
+        <origin rpy="1.5708 0 1.5708" xyz="0.032879 0 0.0105"/>
+        <parent link="bota_ft_sensor_mounting"/>
+        <child link="bota_ft_sensor_mech3"/>
+      </joint>
+      <link name="bota_ft_sensor_mech3"/>
     </xacro:unless>
     <xacro:if value="${hand and ee_id == 'franka_hand'}">
@@ -80,5 +126,5 @@
         <xacro:property name="ee_color" value="white" />
       </xacro:if>
-      <xacro:property name="connection" value="${special_connection if special_connection != '' else robot_type + '_link8'}" />
+      <xacro:property name="connection" value="${'bota_ft_sensor_wrench' if special_connection != '' else robot_type + '_link8'}" />
       <xacro:franka_hand
         connected_to="${arm_prefix}${connection}"
@@ -100,5 +146,5 @@
       <xacro:include filename="$(find cho_franka_description)/end_effectors/common/ee_with_one_link.xacro"/>
       <xacro:include filename="$(find cho_franka_description)/end_effectors/common/utils.xacro" />
-      <xacro:property name="connection" value="${special_connection if special_connection != '' else robot_type + '_link8'}" />
+      <xacro:property name="connection" value="${'bota_ft_sensor_wrench' if special_connection != '' else robot_type + '_link8'}" />
       <xacro:ee_with_one_link
         connected_to="${arm_prefix}${connection}"

File: cho_robots_description/cho_franka_description/urdf/fr3_with_ft_sensor/fr3_franka_hand.urdf (robot description, URDF)
Before this commit: robot fr3, 36 links, 35 joints
Links:
- removed link ft_sensor
- added link bota_ft_sensor_mech1
- added link bota_ft_sensor_mech2
- added link bota_ft_sensor_mech3
- added link bota_ft_sensor_mounting, mass 0.15393; collision cylinder length=0.01 radius=0.0315; collision cylinder length=0.028 radius=0.035
- added link bota_ft_sensor_wrench, mass 0.08253
Joints:
- removed joint flange_to_ft_sensor
- added joint bota_ft_sensor_mounting_to_mech1: type fixed, parent bota_ft_sensor_mounting, child bota_ft_sensor_mech1, origin xyz=-0.032879 0 0.0105 rpy=1.5625 0 -1.5708
- added joint bota_ft_sensor_mounting_to_mech2: type fixed, parent bota_ft_sensor_mounting, child bota_ft_sensor_mech2, origin xyz=0 -0.032879 0.0105 rpy=1.5708 0 0
- added joint bota_ft_sensor_mounting_to_mech3: type fixed, parent bota_ft_sensor_mounting, child bota_ft_sensor_mech3, origin xyz=0.032879 0 0.0105 rpy=1.5708 0 1.5708
- added joint bota_ft_sensor_mounting_to_wrench: type fixed, parent bota_ft_sensor_mounting, child bota_ft_sensor_wrench, origin xyz=0 0 0.035 rpy=0 0 0
- added joint robot_mounting_link_to_bota_ft_sensor: type fixed, parent fr3_link8, child bota_ft_sensor_mounting, origin xyz=0 0 0 rpy=0 0 0
- joint fr3_hand_joint: origin xyz=0 0 0.0175 rpy=0 0 -0.7853981633974483 -> xyz=0 0 0 rpy=0 0 -0.7853981633974483; parent ft_sensor -> bota_ft_sensor_wrench
