Commit message: modified:   cho_controller/cho_controller_ur/include/cho_controller_ur/servers/joint_space_action_server.hpp 	modified:   cho_controller/cho_controller_ur/src/base_controller.cpp 	modified:   cho_controller/cho_controller_ur/src/joint_space_controller.cpp 	modified:   cho_controller/cho_controller_ur/src/servers/joint_space_action_server.cpp 	modified:   cho_controller/cho_controller_ur/src/servers/task_space_action_server.cpp 	modified:   cho_robots_bringup/cho_ur_bringup/config/gz/controllers.yaml 	new file:   cho_robots_bringup/cho_ur_bringup/config/mujoco/controllers.yaml 	modified:   cho_robots_bringup/cho_ur_bringup/launch/bringup_gz_robot.launch.py 	new file:   cho_robots_bringup/cho_ur_bringup/launch/bringup_mujoco_robot.launch.py 	modified:   cho_robots_bringup/cho_ur_bringup/package.xml 	modified:   cho_robots_description/cho_ur_description/CMakeLists.txt 	modified:   cho_robots_description/cho_ur_description/package.xml 	modified:   cho_robots_description/cho_ur_description/urdf/ur.urdf.xacro 	new file:   cho_robots_description/cho_ur_description/urdf/ur5e.urdf 	new file:   cho_robots_description/cho_ur_description/xml/CHANGELOG.md 	new file:   cho_robots_description/cho_ur_description/xml/LICENSE 	new file:   cho_robots_description/cho_ur_description/xml/README.md 	new file:   cho_robots_description/cho_ur_description/xml/assets/base_0.obj 	new file:   cho_robots_description/cho_ur_description/xml/assets/base_1.obj 	new file:   cho_robots_description/cho_ur_description/xml/assets/forearm_0.obj 	new file:   cho_robots_description/cho_ur_description/xml/assets/forearm_1.obj 	new file:   cho_robots_description/cho_ur_description/xml/assets/forearm_2.obj 	new file:   cho_robots_description/cho_ur_description/xml/assets/forearm_3.obj 	new file:   cho_robots_description/cho_ur_description/xml/assets/shoulder_0.obj 	new file:   cho_robots_description/cho_ur_description/xml/assets/shoulder_1.obj 	new file:   cho_robots_description/cho_ur_description/xml/assets/shoulder_2.obj 	new file:   cho_robots_description/cho_ur_description/xml/assets/upperarm_0.obj 	new file:   cho_robots_description/cho_ur_description/xml/assets/upperarm_1.obj 	new file:   cho_robots_description/cho_ur_description/xml/assets/upperarm_2.obj 	new file:   cho_robots_description/cho_ur_description/xml/assets/upperarm_3.obj 	new file:   cho_robots_description/cho_ur_description/xml/assets/wrist1_0.obj 	new file:   cho_robots_description/cho_ur_description/xml/assets/wrist1_1.obj 	new file:   cho_robots_description/cho_ur_description/xml/assets/wrist1_2.obj 	new file:   cho_robots_description/cho_ur_description/xml/assets/wrist2_0.obj 	new file:   cho_robots_description/cho_ur_description/xml/assets/wrist2_1.obj 	new file:   cho_robots_description/cho_ur_description/xml/assets/wrist2_2.obj 	new file:   cho_robots_description/cho_ur_description/xml/assets/wrist3.obj 	new file:   cho_robots_description/cho_ur_description/xml/scene.xml 	new file:   cho_robots_description/cho_ur_description/xml/ur5e.png 	new file:   cho_robots_description/cho_ur_description/xml/ur5e.xml 	modified:   cho_task_manager/package.xml 	modified:   cho_task_manager/python/action_client.py

File: cho_robots_description/cho_ur_description/urdf/ur.urdf.xacro (robot description, xacro)
@@ -5,4 +5,6 @@
    <!-- import main macro -->
    <xacro:include filename="$(find cho_ur_description)/urdf/ur_macro.xacro"/>
+   <xacro:include filename="$(find robotiq_description)/urdf/ur_to_robotiq_adapter.urdf.xacro"/>
+   <xacro:include filename="$(find robotiq_description)/urdf/robotiq_2f_85_macro.urdf.xacro"/>
    <!-- possible 'ur_type' values: ur3, ur5, ur10, ur3e, ur5e, ur7e, ur10e, ur12e, ur16e, ur8long, ur15, ur18, ur20, ur30 -->
    <!-- the default value should raise an error in case this was called without defining the type -->
@@ -45,4 +47,5 @@
    <xacro:arg name="sim_ignition" default="false" />
    <xacro:arg name="simulation_controllers" default="" />
+   <xacro:arg name="load_gripper" default="false" />
    <!-- initial position for simulations (Fake Hardware, Gazebo, Ignition) -->
    <xacro:arg name="initial_positions_file" default="$(find cho_ur_description)/config/initial_positions.yaml"/>
@@ -117,4 +120,16 @@
      <origin xyz="0 0 0" rpy="0 0 0" />          <!-- position robot in the world -->
    </xacro:ur_robot>
+   <xacro:if value="$(arg load_gripper)">
+     <xacro:ur_to_robotiq prefix="$(arg tf_prefix)" connected_to="$(arg tf_prefix)tool0">
+     </xacro:ur_to_robotiq>
+     <xacro:robotiq_gripper
+       name="$(arg tf_prefix)robotiq_gripper"
+       prefix="$(arg tf_prefix)"
+       parent="$(arg tf_prefix)gripper_mount_link"
+       sim_ignition="$(arg sim_ignition)"
+       use_fake_hardware="$(arg use_fake_hardware)">
+       <origin xyz="0 0 0" rpy="0 0 0"/>
+     </xacro:robotiq_gripper>
+   </xacro:if>
    <xacro:if value="$(arg sim_gazebo)">
     <!-- Gazebo plugins -->
