Commit message: modified:   AGENTS.md 	modified:   CLAUDE.md 	modified:   README.md 	modified:   cho_bringup/cho_bringup_franka/CMakeLists.txt 	modified:   cho_bringup/cho_bringup_franka/launch/bringup_gz_robot.launch.py 	modified:   cho_bringup/cho_bringup_franka/launch/bringup_mujoco_robot.launch.py 	modified:   cho_bringup/cho_bringup_franka/launch/bringup_real_robot.launch.py 	modified:   cho_bringup/cho_bringup_franka/package.xml 	modified:   cho_bringup/cho_bringup_franka/scripts/mock_franka_gripper.py 	modified:   cho_bringup/cho_bringup_franka/utils/launch_utils.py 	modified:   cho_bringup/cho_bringup_ur/CMakeLists.txt 	modified:   cho_bringup/cho_bringup_ur/launch/bringup_gz_robot.launch.py 	modified:   cho_bringup/cho_bringup_ur/launch/bringup_mujoco_robot.launch.py 	modified:   cho_bringup/cho_bringup_ur/launch/bringup_real_robot.launch.py 	modified:   cho_bringup/cho_bringup_ur/package.xml 	modified:   cho_controller/cho_controller_franka/src/gripper_controller.cpp 	modified:   cho_description/cho_description_franka/CMakeLists.txt 	modified:   cho_description/cho_description_franka/end_effectors/cobot_pump/cobot_pump.urdf.xacro 	modified:   cho_description/cho_description_franka/end_effectors/cobot_pump/cobot_pump_arguments.xacro 	modified:   cho_description/cho_description_franka/end_effectors/common/ee_with_one_link.xacro 	modified:   cho_description/cho_description_franka/end_effectors/common/franka_hand.xacro 	modified:   cho_description/cho_description_franka/end_effectors/common/utils.xacro 	modified:   cho_description/cho_description_franka/end_effectors/franka_hand/franka_hand.urdf.xacro 	modified:   cho_description/cho_description_franka/end_effectors/franka_hand/franka_hand_arguments.xacro 	modified:   cho_description/cho_description_franka/package.xml 	modified:   cho_description/cho_description_franka/robots/common/franka_arm.ros2_control.xacro 	modified:   cho_description/cho_description_franka/robots/common/franka_arm.srdf.xacro 	modified:   cho_description/cho_description_franka/robots/common/franka_arm.xacro 	modified:   cho_description/cho_description_franka/robots/common/franka_robot.xacro 	modified:   cho_description/cho_description_franka/robots/common/utils.xacro 	modified:   cho_description/cho_description_franka/robots/fr3/fr3.srdf.xacro 	modified:   cho_description/cho_description_franka/robots/fr3/fr3.urdf.xacro 	modified:   cho_description/cho_description_franka/urdf/fr3/fr3_franka_hand.urdf 	modified:   cho_description/cho_description_franka/urdf/fr3_with_ft_sensor/fr3_franka_hand.urdf 	modified:   cho_description/cho_description_ur/CMakeLists.txt 	modified:   cho_description/cho_description_ur/config/ur10/visual_parameters.yaml 	modified:   cho_description/cho_description_ur/config/ur10e/visual_parameters.yaml 	modified:   cho_description/cho_description_ur/config/ur12e/visual_parameters.yaml 	modified:   cho_description/cho_description_ur/config/ur15/visual_parameters.yaml 	modified:   cho_description/cho_description_ur/config/ur16e/visual_parameters.yaml 	modified:   cho_description/cho_description_ur/config/ur18/visual_parameters.yaml 	modified:   cho_description/cho_description_ur/config/ur20/visual_parameters.yaml 	modified:   cho_description/cho_description_ur/config/ur3/visual_parameters.yaml 	modified:   cho_description/cho_description_ur/config/ur30/visual_parameters.yaml 	modified:   cho_description/cho_description_ur/config/ur3e/visual_parameters.yaml 	modified:   cho_description/cho_description_ur/config/ur5/visual_parameters.yaml 	modified:   cho_description/cho_description_ur/config/ur5e/visual_parameters.yaml 	modified:   cho_description/cho_description_ur/config/ur7e/visual_parameters.yaml 	modified:   cho_description/cho_description_ur/config/ur8long/visual_parameters.yaml 	modified:   cho_description/cho_description_ur/launch/view_ur.launch.py 	modified:   cho_description/cho_description_ur/launch/view_ur.launch.xml 	modified:   cho_description/cho_description_ur/launch/visualize_ur5e.launch.py 	modified:   cho_description/cho_description_ur/package.xml 	modified:   cho_description/cho_description_ur/test/test_ur_urdf_xacro.py 	modified:   cho_description/cho_description_ur/test/test_view_ur_launch.py 	modified:   cho_description/cho_description_ur/urdf/ur.urdf.xacro 	modified:   cho_description/cho_description_ur/urdf/ur5e.urdf 	modified:   cho_description/cho_description_ur/urdf/ur_macro.xacro 	new file:   cho_robots_description/cho_ur_description/xml/ur5e.xml 	modified:   cho_task_manager/cho_task_manager/task_manager_node.py 	modified:   cho_task_manager/cho_task_manager/tasks/__init__.py 	new file:   cho_task_manager/cho_task_manager/tasks/franka/__init__.py 	new file:   cho_task_manager/cho_task_manager/tasks/franka/forge.py 	new file:   cho_task_manager/cho_task_manager/tasks/franka/pick_and_place.py 	new file:   cho_task_manager/cho_task_manager/tasks/ur/__init__.py 	new file:   cho_task_manager/cho_task_manager/tasks/ur/multi_move.py 	new file:   cho_task_manager/cho_task_manager/tasks/ur/pick_and_place.py 	modified:   cho_task_manager/cho_task_manager/utils/controller_names.py 	modified:   cho_task_manager/config/robots/franka.yaml 	modified:   cho_task_manager/config/robots/ur5e.yaml

File: cho_description/cho_description_franka/end_effectors/cobot_pump/cobot_pump.urdf.xacro (robot description, xacro)
@@ -1,11 +1,11 @@
 <?xml version="1.0" encoding="utf-8"?>
 <robot xmlns:xacro="http://www.ros.org/wiki/xacro" name="cobot_pump">
-  <xacro:include filename="$(find cho_franka_description)/end_effectors/common/utils.xacro" />
-  <xacro:include filename="$(find cho_franka_description)/end_effectors/common/ee_with_one_link.xacro"/>
-  <xacro:include filename="$(find cho_franka_description)/end_effectors/cobot_pump/cobot_pump_arguments.xacro"/>
+  <xacro:include filename="$(find cho_description_franka)/end_effectors/common/utils.xacro" />
+  <xacro:include filename="$(find cho_description_franka)/end_effectors/common/ee_with_one_link.xacro"/>
+  <xacro:include filename="$(find cho_description_franka)/end_effectors/cobot_pump/cobot_pump_arguments.xacro"/>
   <xacro:ee_with_one_link connected_to="$(arg special_connection)"
                           robot_type="$(arg robot_type)"
                           ee_id="$(arg ee_id)"
-                          ee_inertials="${xacro.load_yaml('$(find cho_franka_description)/end_effectors/$(arg ee_id)/inertials.yaml')}"
+                          ee_inertials="${xacro.load_yaml('$(find cho_description_franka)/end_effectors/$(arg ee_id)/inertials.yaml')}"
                           rpy_ee="$(arg rpy_ee)"
                           xyz_ee="$(arg xyz_ee)"

File: cho_description/cho_description_franka/end_effectors/cobot_pump/cobot_pump_arguments.xacro (robot description, xacro)
@@ -22,4 +22,4 @@
   <xacro:arg name="gazebo" default="false" />
   <!-- Name of the description package -->
-  <xacro:arg name="description_pkg" default="cho_franka_description" />
+  <xacro:arg name="description_pkg" default="cho_description_franka" />
 </robot>

File: cho_description/cho_description_franka/end_effectors/common/ee_with_one_link.xacro (robot description, xacro)
@@ -2,5 +2,5 @@
 <robot xmlns:xacro="http://www.ros.org/wiki/xacro" name="ee_with_one_link">
   <!-- safety_distance: Minimum safety distance in [m] by which the collision volumes are expanded and which is enforced during robot motions -->
-  <xacro:macro name="ee_with_one_link" params="connected_to:='' robot_type arm_prefix:='' ee_id ee_inertials rpy_ee:='0 0 0' xyz_ee:='0 0 0' tcp_xyz:='0 0 0' tcp_rpy:='0 0 0' safety_distance:=0 gazebo:=false description_pkg:=cho_franka_description with_sc:=false">
+  <xacro:macro name="ee_with_one_link" params="connected_to:='' robot_type arm_prefix:='' ee_id ee_inertials rpy_ee:='0 0 0' xyz_ee:='0 0 0' tcp_xyz:='0 0 0' tcp_rpy:='0 0 0' safety_distance:=0 gazebo:=false description_pkg:=cho_description_franka with_sc:=false">
     <xacro:property name="ee_prefix" default="robot_"/>
     <xacro:unless value="${robot_type == ''}">

File: cho_description/cho_description_franka/end_effectors/common/franka_hand.xacro (robot description, xacro)
@@ -12,5 +12,5 @@
                        safety_distance:=0
                        gazebo:=false
-                       description_pkg:=cho_franka_description
+                       description_pkg:=cho_description_franka
                        with_sc:=false
                        no_prefix:=false">

File: cho_description/cho_description_franka/end_effectors/common/utils.xacro (robot description, xacro)
@@ -42,5 +42,5 @@
       <collision name="${prefix}${name}_collision">
         <geometry>
-          <mesh filename="package://cho_franka_description/meshes/robot_ee/${ee_id}/collision/${name}.stl" />
+          <mesh filename="package://cho_description_franka/meshes/robot_ee/${ee_id}/collision/${name}.stl" />
         </geometry>
       </collision>

File: cho_description/cho_description_franka/end_effectors/franka_hand/franka_hand.urdf.xacro (robot description, xacro)
@@ -1,11 +1,11 @@
 <?xml version="1.0" encoding="utf-8"?>
 <robot xmlns:xacro="http://www.ros.org/wiki/xacro" name="franka_hand">
-  <xacro:include filename="$(find cho_franka_description)/end_effectors/common/utils.xacro" />
-  <xacro:include filename="$(find cho_franka_description)/end_effectors/common/franka_hand.xacro"/>
-  <xacro:include filename="$(find cho_franka_description)/end_effectors/franka_hand/franka_hand_arguments.xacro"/>
+  <xacro:include filename="$(find cho_description_franka)/end_effectors/common/utils.xacro" />
+  <xacro:include filename="$(find cho_description_franka)/end_effectors/common/franka_hand.xacro"/>
+  <xacro:include filename="$(find cho_description_franka)/end_effectors/franka_hand/franka_hand_arguments.xacro"/>
   <xacro:franka_hand connected_to="$(arg special_connection)"
                      robot_type="$(arg robot_type)"
                      ee_id="$(arg ee_id)_$(arg ee_color)"
-                     ee_inertials="${xacro.load_yaml('$(find cho_franka_description)/end_effectors/$(arg ee_id)/inertials.yaml')}"
+                     ee_inertials="${xacro.load_yaml('$(find cho_description_franka)/end_effectors/$(arg ee_id)/inertials.yaml')}"
                      rpy_ee="$(arg rpy_ee)"
                      xyz_ee="$(arg xyz_ee)"

File: cho_description/cho_description_franka/end_effectors/franka_hand/franka_hand_arguments.xacro (robot description, xacro)
@@ -24,4 +24,4 @@
   <xacro:arg name="gazebo" default="false" />
   <!-- Name of the description package -->
-  <xacro:arg name="description_pkg" default="cho_franka_description" />
+  <xacro:arg name="description_pkg" default="cho_description_franka" />
 </robot>

File: cho_description/cho_description_franka/robots/common/franka_arm.ros2_control.xacro (robot description, xacro)
@@ -96,5 +96,5 @@
       <gazebo>
         <plugin filename="franka_ign_ros2_control-system" name="ign_ros2_control::IgnitionROS2ControlPlugin">
-          <parameters>$(find cho_franka_bringup)/config/gazebo/controllers.yaml</parameters>
+          <parameters>$(find cho_bringup_franka)/config/gazebo/controllers.yaml</parameters>
         </plugin>
       </gazebo>

File: cho_description/cho_description_franka/robots/common/franka_arm.srdf.xacro (robot description, xacro)
@@ -3,5 +3,5 @@
     <xacro:macro name="franka_arm_srdf" params="robot_type hand:='true' ee_id:=franka_hand arm_prefix='' no_prefix='false'">
         <xacro:property name="prefix" value="${'' if no_prefix else arm_prefix + robot_type + '_'}" />
-        <xacro:include filename="$(find cho_franka_description)/robots/common/group_definition.xacro"/>
+        <xacro:include filename="$(find cho_description_franka)/robots/common/group_definition.xacro"/>
         <xacro:property name="tip_link" value="${prefix + 'hand_tcp' if hand and ee_id == 'franka_hand' else prefix + 'link8'}"/>
         <xacro:group_definition prefix="${prefix}" group_name="${prefix}arm" tip_link="${tip_link}"/>
@@ -32,5 +32,5 @@
         <xacro:if value="${hand}">
             <xacro:if value="${ee_id == 'franka_hand'}">
-                <xacro:include filename="$(find cho_franka_description)/end_effectors/franka_hand/franka_hand.srdf.xacro"/>
+                <xacro:include filename="$(find cho_description_franka)/end_effectors/franka_hand/franka_hand.srdf.xacro"/>
                 <xacro:franka_hand_srdf prefix="${prefix}"/>
             </xacro:if>

File: cho_description/cho_description_franka/robots/common/franka_arm.xacro (robot description, xacro)
@@ -1,12 +1,12 @@
 <?xml version='1.0' encoding='utf-8'?>
 <robot xmlns:xacro="http://www.ros.org/wiki/xacro" name="franka_arm">
-  <xacro:include filename="$(find cho_franka_description)/robots/common/utils.xacro" />
+  <xacro:include filename="$(find cho_description_franka)/robots/common/utils.xacro" />
   <!-- safety_distance: Minimum safety distance in [m] by which the collision volumes are expanded and which is enforced during robot motions -->
   <!-- robot_type: Namespace of the robot arm. Serves to differentiate between arms in case of multiple instances. -->
-  <!-- joint_limits: description of the joint limits that comes from a YAML file. Example definition: ${xacro.load_yaml('$(find cho_franka_description)/robots/fr3/joint_limits.yaml')} -->
-  <!-- kinematics: description of the kinematics that comes from a YAML file. Example definition: ${xacro.load_yaml('$(find cho_franka_description)/robots/fr3/kinematics.yaml')} -->
-  <!-- inertials: description of the inertials that comes from a YAML file. Example definition: ${xacro.load_yaml('$(find cho_franka_description)/robots/fr3/inertials.yaml')} -->
-  <!-- dynamics: description of the dynamics that comes from a YAML file. Example definition: ${xacro.load_yaml('$(find cho_franka_description)/robots/fr3/dynamics.yaml')} -->
-  <xacro:macro name="franka_arm" params="robot_type arm_prefix:='' no_prefix:=false description_pkg:='cho_franka_description' connected_to:='base' xyz:='0 0 0' rpy:='0 0 0' gazebo:='false' safety_distance:=0 joint_limits inertials kinematics accelerometer_config dynamics with_sc:=false" >
+  <!-- joint_limits: description of the joint limits that comes from a YAML file. Example definition: ${xacro.load_yaml('$(find cho_description_franka)/robots/fr3/joint_limits.yaml')} -->
+  <!-- kinematics: description of the kinematics that comes from a YAML file. Example definition: ${xacro.load_yaml('$(find cho_description_franka)/robots/fr3/kinematics.yaml')} -->
+  <!-- inertials: description of the inertials that comes from a YAML file. Example definition: ${xacro.load_yaml('$(find cho_description_franka)/robots/fr3/inertials.yaml')} -->
+  <!-- dynamics: description of the dynamics that comes from a YAML file. Example definition: ${xacro.load_yaml('$(find cho_description_franka)/robots/fr3/dynamics.yaml')} -->
+  <xacro:macro name="franka_arm" params="robot_type arm_prefix:='' no_prefix:=false description_pkg:='cho_description_franka' connected_to:='base' xyz:='0 0 0' rpy:='0 0 0' gazebo:='false' safety_distance:=0 joint_limits inertials kinematics accelerometer_config dynamics with_sc:=false" >
     <!-- Define a property that defaults to 'arm_prefix_robot_type' concatenated with an underscore if 'no_prefix' is not set -->
     <xacro:property name="prefix" value="${'' if no_prefix else arm_prefix + robot_type + '_'}" />

File: cho_description/cho_description_franka/robots/common/franka_robot.xacro (robot description, xacro)
@@ -28,8 +28,8 @@
                       no_prefix:='false'
                       arm_prefix:=''
-                      description_pkg:='cho_franka_description'
+                      description_pkg:='cho_description_franka'
                       connected_to:='base'">
-    <xacro:include filename="$(find cho_franka_description)/robots/common/utils.xacro" />
-    <xacro:include filename="$(find cho_franka_description)/robots/common/franka_arm.xacro" />
+    <xacro:include filename="$(find cho_description_franka)/robots/common/utils.xacro" />
+    <xacro:include filename="$(find cho_description_franka)/robots/common/franka_arm.xacro" />
     <xacro:franka_arm
       robot_type="${robot_type}"
@@ -65,5 +65,5 @@
           <origin rpy="0 0 0" xyz="0 0 0"/>
           <geometry>
-            <mesh filename="package://cho_franka_description/meshes/accessories/ft_sensor/mounting.stl"/>
+            <mesh filename="package://cho_description_franka/meshes/accessories/ft_sensor/mounting.stl"/>
           </geometry>
           <material name="bota_ft_material">
@@ -118,6 +118,6 @@
     </xacro:unless>
     <xacro:if value="${hand and ee_id == 'franka_hand'}">
-      <xacro:include filename="$(find cho_franka_description)/end_effectors/common/franka_hand.xacro"/>
-      <xacro:include filename="$(find cho_franka_description)/end_effectors/common/utils.xacro" />
+      <xacro:include filename="$(find cho_description_franka)/end_effectors/common/franka_hand.xacro"/>
+      <xacro:include filename="$(find cho_description_franka)/end_effectors/common/utils.xacro" />
       <xacro:if value="${robot_type == 'fp3'}">
         <xacro:property name="ee_color" value="black" />
@@ -132,5 +132,5 @@
         arm_prefix="${arm_prefix}"
         ee_id="${ee_id}_${ee_color}"
-        ee_inertials="${xacro.load_yaml('$(find cho_franka_description)/end_effectors/' + ee_id + '/inertials.yaml')}"
+        ee_inertials="${xacro.load_yaml('$(find cho_description_franka)/end_effectors/' + ee_id + '/inertials.yaml')}"
         rpy_ee="${rpy_ee}"
         xyz_ee="${xyz_ee}"
@@ -144,6 +144,6 @@
     </xacro:if>
     <xacro:if value="${hand and ee_id != 'none' and ee_id != 'franka_hand'}">
-      <xacro:include filename="$(find cho_franka_description)/end_effectors/common/ee_with_one_link.xacro"/>
-      <xacro:include filename="$(find cho_franka_description)/end_effectors/common/utils.xacro" />
+      <xacro:include filename="$(find cho_description_franka)/end_effectors/common/ee_with_one_link.xacro"/>
+      <xacro:include filename="$(find cho_description_franka)/end_effectors/common/utils.xacro" />
       <xacro:property name="connection" value="${'bota_ft_sensor_wrench' if special_connection != '' else robot_type + '_link8'}" />
       <xacro:ee_with_one_link
@@ -152,5 +152,5 @@
         arm_prefix="${arm_prefix}"
         ee_id="${ee_id}"
-        ee_inertials="${xacro.load_yaml('$(find cho_franka_description)/end_effectors/' + ee_id + '/inertials.yaml')}"
+        ee_inertials="${xacro.load_yaml('$(find cho_description_franka)/end_effectors/' + ee_id + '/inertials.yaml')}"
         rpy_ee="${rpy_ee}"
         xyz_ee="${xyz_ee}"
@@ -211,5 +211,5 @@
     </xacro:if>
     <xacro:if value="${ros2_control}">
-      <xacro:include filename="$(find cho_franka_description)/robots/common/franka_arm.ros2_control.xacro"/>
+      <xacro:include filename="$(find cho_description_franka)/robots/common/franka_arm.ros2_control.xacro"/>
       <xacro:franka_arm_ros2_control
           robot_type="${robot_type}"

File: cho_description/cho_description_franka/robots/common/utils.xacro (robot description, xacro)
@@ -43,5 +43,5 @@
       <collision name="${prefix}${name}_collision">
         <geometry>
-          <mesh filename="package://cho_franka_description/meshes/robots/${robot_type}/collision/${name}.stl" />
+          <mesh filename="package://cho_description_franka/meshes/robots/${robot_type}/collision/${name}.stl" />
         </geometry>
       </collision>

File: cho_description/cho_description_franka/robots/fr3/fr3.srdf.xacro (robot description, xacro)
@@ -1,5 +1,5 @@
 <?xml version='1.0' encoding='utf-8'?>
 <robot xmlns:xacro="http://www.ros.org/wiki/xacro" name="fr3">
-  <xacro:include filename="$(find cho_franka_description)/robots/common/franka_arm.srdf.xacro"/>
+  <xacro:include filename="$(find cho_description_franka)/robots/common/franka_arm.srdf.xacro"/>
   <!-- The ID of the robot model to be used -->
   <xacro:arg name="robot_type" default="fr3" />

File: cho_description/cho_description_franka/robots/fr3/fr3.urdf.xacro (robot description, xacro)
@@ -1,5 +1,5 @@
 <?xml version='1.0' encoding='utf-8'?>
 <robot xmlns:xacro="http://www.ros.org/wiki/xacro" name="fr3">
-  <xacro:include filename="$(find cho_franka_description)/robots/common/franka_robot.xacro"/>
+  <xacro:include filename="$(find cho_description_franka)/robots/common/franka_robot.xacro"/>
   <!-- Define arguments -->
   <!-- The ID of the robot model to be used -->
@@ -40,14 +40,14 @@
   <xacro:arg name="gazebo_effort" default="false" />
   <!-- Name of the description package -->
-  <xacro:arg name="description_pkg" default="cho_franka_description" />
+  <xacro:arg name="description_pkg" default="cho_description_franka" />
   <!-- Append an underscore to the user-provided prefix, if non-empty. -->
   <xacro:property name="prefix" value="$(arg arm_prefix)"/>
   <xacro:property name="modified_prefix" value="${prefix + '_' if prefix else ''}"/>
   <xacro:franka_robot robot_type="fr3"
-                      joint_limits="${xacro.load_yaml('$(find cho_franka_description)/robots/fr3/joint_limits.yaml')}"
-                      inertials="${xacro.load_yaml('$(find cho_franka_description)/robots/fr3/inertials.yaml')}"
-                      kinematics="${xacro.load_yaml('$(find cho_franka_description)/robots/fr3/kinematics.yaml')}"
-                      accelerometer_config="${xacro.load_yaml('$(find cho_franka_description)/robots/fr3/accelerometers.yaml')}"
-                      dynamics="${xacro.load_yaml('$(find cho_franka_description)/robots/fr3/dynamics.yaml')}"
+                      joint_limits="${xacro.load_yaml('$(find cho_description_franka)/robots/fr3/joint_limits.yaml')}"
+                      inertials="${xacro.load_yaml('$(find cho_description_franka)/robots/fr3/inertials.yaml')}"
+                      kinematics="${xacro.load_yaml('$(find cho_description_franka)/robots/fr3/kinematics.yaml')}"
+                      accelerometer_config="${xacro.load_yaml('$(find cho_description_franka)/robots/fr3/accelerometers.yaml')}"
+                      dynamics="${xacro.load_yaml('$(find cho_description_franka)/robots/fr3/dynamics.yaml')}"
                       gazebo="$(arg gazebo)"
                       hand="$(arg hand)"
