Commit message: modified:   AGENTS.md 	modified:   CLAUDE.md 	modified:   README.md 	modified:   cho_bringup/cho_bringup_franka/CMakeLists.txt 	modified:   cho_bringup/cho_bringup_franka/launch/bringup_gz_robot.launch.py 	modified:   cho_bringup/cho_bringup_franka/launch/bringup_mujoco_robot.launch.py 	modified:   cho_bringup/cho_bringup_franka/launch/bringup_real_robot.launch.py 	modified:   cho_bringup/cho_bringup_franka/package.xml 	modified:   cho_bringup/cho_bringup_franka/scripts/mock_franka_gripper.py 	modified:   cho_bringup/cho_bringup_franka/utils/launch_utils.py 	modified:   cho_bringup/cho_bringup_ur/CMakeLists.txt 	modified:   cho_bringup/cho_bringup_ur/launch/bringup_gz_robot.launch.py 	modified:   cho_bringup/cho_bringup_ur/launch/bringup_mujoco_robot.launch.py 	modified:   cho_bringup/cho_bringup_ur/launch/bringup_real_robot.launch.py 	modified:   cho_bringup/cho_bringup_ur/package.xml 	modified:   cho_controller/cho_controller_franka/src/gripper_controller.cpp 	modified:   cho_description/cho_description_franka/CMakeLists.txt 	modified:   cho_description/cho_description_franka/end_effectors/cobot_pump/cobot_pump.urdf.xacro 	modified:   cho_description/cho_description_franka/end_effectors/cobot_pump/cobot_pump_arguments.xacro 	modified:   cho_description/cho_description_franka/end_effectors/common/ee_with_one_link.xacro 	modified:   cho_description/cho_description_franka/end_effectors/common/franka_hand.xacro 	modified:   cho_description/cho_description_franka/end_effectors/common/utils.xacro 	modified:   cho_description/cho_description_franka/end_effectors/franka_hand/franka_hand.urdf.xacro 	modified:   cho_description/cho_description_franka/end_effectors/franka_hand/franka_hand_arguments.xacro 	modified:   cho_description/cho_description_franka/package.xml 	modified:   cho_description/cho_description_franka/robots/common/franka_arm.ros2_control.xacro 	modified:   cho_description/cho_description_franka/robots/common/franka_arm.srdf.xacro 	modified:   cho_description/cho_description_franka/robots/common/franka_arm.xacro 	modified:   cho_description/cho_description_franka/robots/common/franka_robot.xacro 	modified:   cho_description/cho_description_franka/robots/common/utils.xacro 	modified:   cho_description/cho_description_franka/robots/fr3/fr3.srdf.xacro 	modified:   cho_description/cho_description_franka/robots/fr3/fr3.urdf.xacro 	modified:   cho_description/cho_description_franka/urdf/fr3/fr3_franka_hand.urdf 	modified:   cho_description/cho_description_franka/urdf/fr3_with_ft_sensor/fr3_franka_hand.urdf 	modified:   cho_description/cho_description_ur/CMakeLists.txt 	modified:   cho_description/cho_description_ur/config/ur10/visual_parameters.yaml 	modified:   cho_description/cho_description_ur/config/ur10e/visual_parameters.yaml 	modified:   cho_description/cho_description_ur/config/ur12e/visual_parameters.yaml 	modified:   cho_description/cho_description_ur/config/ur15/visual_parameters.yaml 	modified:   cho_description/cho_description_ur/config/ur16e/visual_parameters.yaml 	modified:   cho_description/cho_description_ur/config/ur18/visual_parameters.yaml 	modified:   cho_description/cho_description_ur/config/ur20/visual_parameters.yaml 	modified:   cho_description/cho_description_ur/config/ur3/visual_parameters.yaml 	modified:   cho_description/cho_description_ur/config/ur30/visual_parameters.yaml 	modified:   cho_description/cho_description_ur/config/ur3e/visual_parameters.yaml 	modified:   cho_description/cho_description_ur/config/ur5/visual_parameters.yaml 	modified:   cho_description/cho_description_ur/config/ur5e/visual_parameters.yaml 	modified:   cho_description/cho_description_ur/config/ur7e/visual_parameters.yaml 	modified:   cho_description/cho_description_ur/config/ur8long/visual_parameters.yaml 	modified:   cho_description/cho_description_ur/launch/view_ur.launch.py 	modified:   cho_description/cho_description_ur/launch/view_ur.launch.xml 	modified:   cho_description/cho_description_ur/launch/visualize_ur5e.launch.py 	modified:   cho_description/cho_description_ur/package.xml 	modified:   cho_description/cho_description_ur/test/test_ur_urdf_xacro.py 	modified:   cho_description/cho_description_ur/test/test_view_ur_launch.py 	modified:   cho_description/cho_description_ur/urdf/ur.urdf.xacro 	modified:   cho_description/cho_description_ur/urdf/ur5e.urdf 	modified:   cho_description/cho_description_ur/urdf/ur_macro.xacro 	new file:   cho_robots_description/cho_ur_description/xml/ur5e.xml 	modified:   cho_task_manager/cho_task_manager/task_manager_node.py 	modified:   cho_task_manager/cho_task_manager/tasks/__init__.py 	new file:   cho_task_manager/cho_task_manager/tasks/franka/__init__.py 	new file:   cho_task_manager/cho_task_manager/tasks/franka/forge.py 	new file:   cho_task_manager/cho_task_manager/tasks/franka/pick_and_place.py 	new file:   cho_task_manager/cho_task_manager/tasks/ur/__init__.py 	new file:   cho_task_manager/cho_task_manager/tasks/ur/multi_move.py 	new file:   cho_task_manager/cho_task_manager/tasks/ur/pick_and_place.py 	modified:   cho_task_manager/cho_task_manager/utils/controller_names.py 	modified:   cho_task_manager/config/robots/franka.yaml 	modified:   cho_task_manager/config/robots/ur5e.yaml

File: cho_description/cho_description_franka/urdf/fr3/fr3_franka_hand.urdf (robot description, URDF)
Before this commit: robot fr3, 35 links, 34 joints
Links:
- link fr3_hand: geometry collision mesh filename=package://cho_description_franka/meshes/robot_ee/franka_han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; visual mesh filename=package://cho_description_franka/meshes/robot_ee/franka_han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
- link fr3_leftfinger: geometry collision box size=17.5e-3 15.2e-3 18.5e-3; collision box size=17.5e-3 7e-3 23.5e-3
- link fr3_link0: geometry collision mesh filename=package://cho_description_franka/meshes/robots/fr3/collisio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; visual mesh filename=package://cho_description_franka/meshes/robots/fr3/visual/l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
- link fr3_link1: geometry collision mesh filename=package://cho_description_franka/meshes/robots/fr3/collisio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; visual mesh filename=package://cho_description_franka/meshes/robots/fr3/visual/l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
- link fr3_link2: geometry collision mesh filename=package://cho_description_franka/meshes/robots/fr3/collisio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; visual mesh filename=package://cho_description_franka/meshes/robots/fr3/visual/l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
- link fr3_link3: geometry collision mesh filename=package://cho_description_franka/meshes/robots/fr3/collisio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; visual mesh filename=package://cho_description_franka/meshes/robots/fr3/visual/l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
- link fr3_link4: geometry collision mesh filename=package://cho_description_franka/meshes/robots/fr3/collisio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; visual mesh filename=package://cho_description_franka/meshes/robots/fr3/visual/l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
- link fr3_link5: geometry collision mesh filename=package://cho_description_franka/meshes/robots/fr3/collisio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; visual mesh filename=package://cho_description_franka/meshes/robots/fr3/visual/l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
- link fr3_link6: geometry collision mesh filename=package://cho_description_franka/meshes/robots/fr3/collisio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; visual mesh filename=package://cho_description_franka/meshes/robots/fr3/visual/l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
- link fr3_link7: geometry collision mesh filename=package://cho_description_franka/meshes/robots/fr3/collisio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; visual mesh filename=package://cho_description_franka/meshes/robots/fr3/visual/l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
- link fr3_rightfinger: geometry collision box size=17.5e-3 15.2e-3 18.5e-3; collision box size=17.5e-3 7e-3 23.5e-3

File: cho_description/cho_description_franka/urdf/fr3_with_ft_sensor/fr3_franka_hand.urdf (robot description, URDF)
Before this commit: robot fr3, 40 links, 39 joints
Links:
- link bota_ft_sensor_mounting: geometry collision cylinder length=0.01 radius=0.0315; collision cylinder length=0.028 radius=0.035
- link fr3_hand: geometry collision mesh filename=package://cho_description_franka/meshes/robot_ee/franka_han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; visual mesh filename=package://cho_description_franka/meshes/robot_ee/franka_han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
- link fr3_leftfinger: geometry collision box size=17.5e-3 15.2e-3 18.5e-3; collision box size=17.5e-3 7e-3 23.5e-3
- link fr3_link0: geometry collision mesh filename=package://cho_description_franka/meshes/robots/fr3/collisio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; visual mesh filename=package://cho_description_franka/meshes/robots/fr3/visual/l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
- link fr3_link1: geometry collision mesh filename=package://cho_description_franka/meshes/robots/fr3/collisio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; visual mesh filename=package://cho_description_franka/meshes/robots/fr3/visual/l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
- link fr3_link2: geometry collision mesh filename=package://cho_description_franka/meshes/robots/fr3/collisio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; visual mesh filename=package://cho_description_franka/meshes/robots/fr3/visual/l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
- link fr3_link3: geometry collision mesh filename=package://cho_description_franka/meshes/robots/fr3/collisio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; visual mesh filename=package://cho_description_franka/meshes/robots/fr3/visual/l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
- link fr3_link4: geometry collision mesh filename=package://cho_description_franka/meshes/robots/fr3/collisio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; visual mesh filename=package://cho_description_franka/meshes/robots/fr3/visual/l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
- link fr3_link5: geometry collision mesh filename=package://cho_description_franka/meshes/robots/fr3/collisio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; visual mesh filename=package://cho_description_franka/meshes/robots/fr3/visual/l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
- link fr3_link6: geometry collision mesh filename=package://cho_description_franka/meshes/robots/fr3/collisio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; visual mesh filename=package://cho_description_franka/meshes/robots/fr3/visual/l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
- link fr3_link7: geometry collision mesh filename=package://cho_description_franka/meshes/robots/fr3/collisio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; visual mesh filename=package://cho_description_franka/meshes/robots/fr3/visual/l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
- link fr3_rightfinger: geometry collision box size=17.5e-3 15.2e-3 18.5e-3; collision box size=17.5e-3 7e-3 23.5e-3

File: cho_description/cho_description_ur/urdf/ur.urdf.xacro (robot description, xacro)
@@ -4,5 +4,5 @@
    <xacro:arg name="name" default="ur"/>
    <!-- import main macro -->
-   <xacro:include filename="$(find cho_ur_description)/urdf/ur_macro.xacro"/>
+   <xacro:include filename="$(find cho_description_ur)/urdf/ur_macro.xacro"/>
    <xacro:include filename="$(find robotiq_description)/urdf/ur_to_robotiq_adapter.urdf.xacro"/>
    <xacro:include filename="$(find robotiq_description)/urdf/robotiq_2f_85_macro.urdf.xacro"/>
@@ -12,8 +12,8 @@
    <!-- parameters -->
    <xacro:arg name="tf_prefix" default="" />
-   <xacro:arg name="joint_limit_params" default="$(find cho_ur_description)/config/$(arg ur_type)/joint_limits.yaml"/>
-   <xacro:arg name="kinematics_params" default="$(find cho_ur_description)/config/$(arg ur_type)/default_kinematics.yaml"/>
-   <xacro:arg name="physical_params" default="$(find cho_ur_description)/config/$(arg ur_type)/physical_parameters.yaml"/>
-   <xacro:arg name="visual_params" default="$(find cho_ur_description)/config/$(arg ur_type)/visual_parameters.yaml"/>
+   <xacro:arg name="joint_limit_params" default="$(find cho_description_ur)/config/$(arg ur_type)/joint_limits.yaml"/>
+   <xacro:arg name="kinematics_params" default="$(find cho_description_ur)/config/$(arg ur_type)/default_kinematics.yaml"/>
+   <xacro:arg name="physical_params" default="$(find cho_description_ur)/config/$(arg ur_type)/physical_parameters.yaml"/>
+   <xacro:arg name="visual_params" default="$(find cho_description_ur)/config/$(arg ur_type)/visual_parameters.yaml"/>
    <xacro:arg name="transmission_hw_interface" default=""/>
    <xacro:arg name="safety_limits" default="false"/>
@@ -49,5 +49,5 @@
    <xacro:arg name="load_gripper" default="false" />
    <!-- initial position for simulations (Fake Hardware, Gazebo, Ignition) -->
-   <xacro:arg name="initial_positions_file" default="$(find cho_ur_description)/config/initial_positions.yaml"/>
+   <xacro:arg name="initial_positions_file" default="$(find cho_description_ur)/config/initial_positions.yaml"/>
    <!-- convert to property to use substitution in function -->
    <xacro:property name="initial_positions_file" default="$(arg initial_positions_file)"/>

File: cho_description/cho_description_ur/urdf/ur5e.urdf (robot description, URDF)
Before this commit: robot ur, 13 links, 12 joints
Links:
- link base_link_inertia: geometry collision mesh filename=package://cho_description_ur/meshes/ur5e/collision/base.stl; visual mesh filename=package://cho_description_ur/meshes/ur5e/visual/base.dae
- link forearm_link: geometry collision mesh filename=package://cho_description_ur/meshes/ur5e/collision/forearm.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; visual mesh filename=package://cho_description_ur/meshes/ur5e/visual/forearm.dae
- link shoulder_link: geometry collision mesh filename=package://cho_description_ur/meshes/ur5e/collision/shoulder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; visual mesh filename=package://cho_description_ur/meshes/ur5e/visual/shoulder.dae
- link upper_arm_link: geometry collision mesh filename=package://cho_description_ur/meshes/ur5e/collision/upperarm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; visual mesh filename=package://cho_description_ur/meshes/ur5e/visual/upperarm.dae
- link wrist_1_link: geometry collision mesh filename=package://cho_description_ur/meshes/ur5e/collision/wrist1.s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; visual mesh filename=package://cho_description_ur/meshes/ur5e/visual/wrist1.dae
- link wrist_2_link: geometry collision mesh filename=package://cho_description_ur/meshes/ur5e/collision/wrist2.s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; visual mesh filename=package://cho_description_ur/meshes/ur5e/visual/wrist2.dae
- link wrist_3_link: geometry collision mesh filename=package://cho_description_ur/meshes/ur5e/collision/wrist3.s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; visual mesh filename=package://cho_description_ur/meshes/ur5e/visual/wrist3.dae

File: cho_description/cho_description_ur/urdf/ur_macro.xacro (robot description, xacro)
@@ -42,6 +42,6 @@
      - Muhammad Asif Rana
   -->
-  <xacro:include filename="$(find cho_ur_description)/urdf/inc/ur_transmissions.xacro" />
-  <xacro:include filename="$(find cho_ur_description)/urdf/inc/ur_common.xacro" />
+  <xacro:include filename="$(find cho_description_ur)/urdf/inc/ur_transmissions.xacro" />
+  <xacro:include filename="$(find cho_description_ur)/urdf/inc/ur_common.xacro" />
   <xacro:macro name="ur_robot" params="
     name
@@ -94,5 +94,5 @@
     <xacro:if value="${generate_ros2_control_tag}">
       <!-- ros2 control include -->
-      <xacro:include filename="$(find cho_ur_description)/urdf/ur.ros2_control.xacro" />
+      <xacro:include filename="$(find cho_description_ur)/urdf/ur.ros2_control.xacro" />
       <!-- ros2 control instance -->
       <xacro:ur_ros2_control
