Commit message: Add MIT OpenArm control stack and robot control tooling

File: cho_description/cho_description_fr5/urdf/fr5.ros2_control.xacro (robot description, xacro)
@@ -32,5 +32,5 @@
     </joint>
   </xacro:macro>
-  <xacro:macro name="fr5_ros2_control" params="name prefix hardware robot_ip initial_positions">
+  <xacro:macro name="fr5_ros2_control" params="name prefix hardware robot_ip initial_positions mujoco_initial_keyframe:=''">
     <ros2_control name="${name}" type="system">
       <hardware>
@@ -38,4 +38,7 @@
           <plugin>mujoco_ros2_control/MujocoSystemInterface</plugin>
           <param name="mujoco_model">$(find cho_description_fr5)/xml/scene.xml</param>
+          <xacro:if value="${bool(mujoco_initial_keyframe)}">
+            <param name="initial_keyframe">${mujoco_initial_keyframe}</param>
+          </xacro:if>
         </xacro:if>
         <xacro:if value="${hardware == 'isaac'}">

File: cho_description/cho_description_fr5/urdf/fr5.urdf.xacro (robot description, xacro)
@@ -15,4 +15,5 @@
   <xacro:arg name="initial_positions_file"
              default="$(find cho_description_fr5)/config/initial_positions.yaml"/>
+  <xacro:arg name="mujoco_initial_keyframe" default=""/>
   <xacro:property name="initial_positions_file" default="$(arg initial_positions_file)"/>
   <xacro:property name="initial_positions" value="${xacro.load_yaml(initial_positions_file)}"/>
@@ -28,5 +29,6 @@
     hardware="$(arg hardware)"
     robot_ip="$(arg robot_ip)"
-    initial_positions="${initial_positions}"/>
+    initial_positions="${initial_positions}"
+    mujoco_initial_keyframe="$(arg mujoco_initial_keyframe)"/>
   <!-- Gazebo (Ignition) ros2_control system plugin. -->
   <xacro:if value="${'$(arg hardware)' == 'gazebo'}">

File: cho_description/cho_description_openarm/robots/openarm_v10/openarm_v10.ros2_control.xacro (robot description, xacro)
@@ -25,4 +25,7 @@
       hardware:=mujoco
       control_mode:=torque
+      mujoco_position_profile:=standard
+      mujoco_mit_prototype:=false
+      mujoco_mit_headless:=false
       bimanual:=false
       arm_prefix:=''
@@ -103,4 +106,9 @@
         </xacro:if>
         <xacro:unless value="${mit_gains}">
+          <xacro:if value="${hardware == 'mujoco' and mujoco_mit_prototype}">
+            <xacro:if value="${gripper}"><command_interface name="position"/></xacro:if>
+            <xacro:unless value="${gripper}"><command_interface name="position"/><command_interface name="velocity"/><command_interface name="stiffness"/><command_interface name="damping"/><command_interface name="effort"/></xacro:unless>
+          </xacro:if>
+          <xacro:unless value="${hardware == 'mujoco' and mujoco_mit_prototype}">
           <!-- The gripper is position-driven in every simulator actuator set
                (its MJCF actuator is a position servo on the "split" tendon in
@@ -123,4 +131,5 @@
               <command_interface name="effort"/>
             </xacro:unless>
+          </xacro:unless>
           </xacro:unless>
         </xacro:unless>
@@ -239,10 +248,24 @@
           </xacro:if>
           <xacro:if value="${hardware == 'mujoco'}">
-            <plugin>mujoco_ros2_control/MujocoSystemInterface</plugin>
+            <xacro:if value="${mujoco_mit_prototype}">
+              <plugin>cho_hardware_openarm_mit_mujoco/MitMujocoSystem</plugin>
+              <param name="mit_safety_profile_file">$(find cho_description_openarm)/config/mit_safety_profiles_v1.yaml</param>
+              <param name="mit_safety_profile">mujoco_sim_safe</param>
+              <param name="mit_expected_update_rate_hz">1000</param>
+              <param name="headless">${mujoco_mit_headless}</param>
+            </xacro:if>
+            <xacro:unless value="${mujoco_mit_prototype}">
+              <plugin>mujoco_ros2_control/MujocoSystemInterface</plugin>
+            </xacro:unless>
             <!-- Pick the actuator set that matches control_mode. MuJoCo writes the
                  raw command into mjData.ctrl with no unit conversion, so a position
                  command sent to a <motor> would be read as a torque. -->
             <xacro:if value="${control_mode == 'position'}">
-              <param name="mujoco_model">$(find cho_description_openarm)/xml/${scene_dir}/scene_position.xml</param>
+              <xacro:if value="${mujoco_position_profile == 'moveit'}">
+                <param name="mujoco_model">$(find cho_description_openarm)/xml/${scene_dir}/scene_position_moveit.xml</param>
+              </xacro:if>
+              <xacro:unless value="${mujoco_position_profile == 'moveit'}">
+                <param name="mujoco_model">$(find cho_description_openarm)/xml/${scene_dir}/scene_position.xml</param>
+              </xacro:unless>
             </xacro:if>
             <xacro:if value="${control_mode == 'velocity'}">
@@ -259,4 +282,14 @@
         <xacro:arm_joints/>
         <xacro:hand_joints/>
+        <xacro:if value="${hardware == 'mujoco' and mujoco_mit_prototype}">
+          <xacro:if value="${bimanual}">
+            <gpio name="openarm_left_arm"><command_interface name="mit_session_echo"/><command_interface name="mit_lease_cycles"/><command_interface name="mit_commit_generation"/><command_interface name="mit_safe_request_generation"/><state_interface name="mit_session_id"/><state_interface name="mit_ack_generation"/><state_interface name="mit_safe_generation"/><state_interface name="mit_safe_ack_generation"/><state_interface name="mit_status"/></gpio>
+            <gpio name="openarm_right_arm"><command_interface name="mit_session_echo"/><command_interface name="mit_lease_cycles"/><command_interface name="mit_commit_generation"/><command_interface name="mit_safe_request_generation"/><state_interface name="mit_session_id"/><state_interface name="mit_ack_generation"/><state_interface name="mit_safe_generation"/><state_interface name="mit_safe_ack_generation"/><state_interface name="mit_status"/></gpio>
+            <gpio name="openarm_bimanual"><command_interface name="mit_pair_ownership"/><state_interface name="mit_pair_stop_ready"/></gpio>
+          </xacro:if>
+          <xacro:unless value="${bimanual}">
+            <gpio name="openarm_arm"><command_interface name="mit_session_echo"/><command_interface name="mit_lease_cycles"/><command_interface name="mit_commit_generation"/><command_interface name="mit_safe_request_generation"/><state_interface name="mit_session_id"/><state_interface name="mit_ack_generation"/><state_interface name="mit_safe_generation"/><state_interface name="mit_safe_ack_generation"/><state_interface name="mit_status"/></gpio>
+          </xacro:unless>
+        </xacro:if>
       </ros2_control>
     </xacro:unless>

File: cho_description/cho_description_openarm/robots/openarm_v10/openarm_v10.urdf.xacro (robot description, xacro)
@@ -32,4 +32,7 @@
   <xacro:arg name="hardware"      default="mujoco"/>
   <xacro:arg name="control_mode"  default="torque"/>
+  <xacro:arg name="mujoco_position_profile" default="standard"/>
+  <xacro:arg name="mujoco_mit_prototype" default="false"/>
+  <xacro:arg name="mujoco_mit_headless" default="false"/>
   <xacro:arg name="bimanual"      default="false"/>
   <xacro:arg name="arm_prefix"    default=""/>
@@ -125,4 +128,7 @@
       hardware="$(arg hardware)"
       control_mode="$(arg control_mode)"
+      mujoco_position_profile="$(arg mujoco_position_profile)"
+      mujoco_mit_prototype="$(arg mujoco_mit_prototype)"
+      mujoco_mit_headless="$(arg mujoco_mit_headless)"
       bimanual="$(arg bimanual)"
       arm_prefix="$(arg arm_prefix)"
