Commit message: Give the FR5's AG-95 a shape, so MoveIt stops planning through it
The gripper was two empty frames. MoveIt therefore collision-checked
nothing where a 200 mm body hangs off the flange, planned as though that
volume were empty, and drove the gripper into the arm.

Geometry comes from ian-chuang/dh_ag95_gripper_ros2 (MIT, vendored under
meshes/ag95 with its licence): the two links that are rigid with respect
to the flange, unmodified. Measured off those meshes in the flange
frame, the static parts occupy x +/-63.5, y +/-33.5, z -3.5 to
+134.5 mm, and the jaws sweep x +/-84.1, y +/-25.4, z +90.4 to
+200.8 mm over the whole stroke. All three collision volumes sit on one
link, because every extra link is another row of MoveIt's collision
matrix for no gain when the parts do not move independently.

The jaws are one box rather than the real linkage. Upstream drives them
as a four-bar per side - one actuated joint plus seven mimic, with the
separation trigonometric in the angle - while cho_controller_gripper
drives ONE joint through a LINEAR width map and the real gripper is
commanded as a stroke percentage, so adopting that linkage would mean
changing a controller contract shared with franka, openarm and ur. A box
sized to the swept volume is conservative in the direction that matters:
it can refuse a plan the real gripper would have cleared, but it cannot
pass one the real gripper would have hit. It is also why the box is
sized from the mesh sweep and not from either available grasp frame,
which disagree - 170 mm in the operator's own fr5_ag95 URDF, 190 mm
upstream.

Where it mounts is confirmed rather than assumed. wrist3_link's own mesh
runs to z = +0.099, so the 100 mm tool_tcp offset is the length of the
wrist and tool_tcp IS the flange face. The operator's URDF mounts the
gripper on a tool0 whose net transform from wrist3_link is (0, 0, 0.1)
with an identity rotation - the same frame - and puts its jaw knuckles
at x = -0.016 and +0.016, so the jaws separate along x. That fixes the
finger axis and makes yaw 0 correct here; the parameter stays for a
gripper bolted on a quarter turn round.

The SRDF gains exactly one disable_collisions pair. The mounting plate
starts 3.5 mm behind the flange face, overlapping the wrist mesh by
2.5 mm permanently, and without the pair MoveIt reports every state as
in collision and nothing plans at all. Only that pair: the gripper
reaching wrist2_link or further back is a real collision at extreme
wrist angles. The SRDF is processed with xacro now, so the pair appears
only when the description actually has the gripper and never dangles.

MuJoCo gets a matching slide joint, actuator and visual geoms, so the
same Gripper action moves something in simulation and the gripper is
visible. Visual-only like every geom in that model, so it still cannot
hold an object. MJCF keyframes are sized by nq and nu, so all three
carry the finger, and the registry guard tests now compare the arm
prefix and pin the finger value instead of demanding six.

Co-Authored-By: Claude Opus 5 <noreply@anthropic.com>

File: cho_description/cho_description_fr5/urdf/fr5.ros2_control.xacro (robot description, xacro)
@@ -32,5 +32,33 @@
     </joint>
   </xacro:macro>
-  <xacro:macro name="fr5_ros2_control" params="name prefix hardware robot_ip initial_positions mujoco_initial_keyframe:=''">
+  <!--
+    On the real robot the AG-95 hangs off the controller's RS485 bus rather than
+    off ros2_control, and FairinoHardwareInterface maps this joint on to the
+    SDK's MoveGripper()/stroke-percentage feedback. There it is position only:
+    the controller reports a stroke percentage and no finger velocity.
+    MuJoCo drives the matching slide joint in xml/fr5.xml instead, and does
+    integrate a velocity, so the simulated build asks for that state too. The
+    other backends have no gripper joint at all - Gazebo and Isaac would need
+    the same modelling done in their own scenes first.
+  -->
+  <xacro:macro name="fr5_gripper_joint" params="joint_name with_velocity:=^|false">
+    <joint name="${joint_name}">
+      <command_interface name="position">
+        <param name="min">0.0</param>
+        <param name="max">0.0475</param>
+      </command_interface>
+      <state_interface name="position"/>
+      <xacro:if value="${with_velocity}">
+        <state_interface name="velocity"/>
+      </xacro:if>
+    </joint>
+  </xacro:macro>
+  <xacro:macro name="fr5_ros2_control" params="name prefix hardware robot_ip initial_positions gripper:='none' gripper_company:='4' gripper_device:='0'
+                      gripper_softversion:='0' gripper_bus:='1' gripper_index:='1'
+                      gripper_speed_percent:='30' gripper_force_percent:='30'
+                      gripper_percent_at_closed:='0' gripper_percent_at_open:='100'
+                      gripper_open_on_activate:='false' gripper_apply_config:='false'
+                      gripper_required:='false'
+                      mujoco_initial_keyframe:=''">
     <ros2_control name="${name}" type="system">
       <hardware>
@@ -58,8 +86,48 @@
         </xacro:if>
         <xacro:if value="${hardware == 'fairino'}">
-          <!-- Real FR5 over libfairino. The fork reads robot_ip from this
-               hardware parameter (the upstream v3_9_9 hardcodes it). -->
+          <!-- Real FR5 over libfairino. The vendored driver is patched to read
+               robot_ip from this hardware parameter (upstream hardcodes it). -->
           <plugin>fairino_hardware/FairinoHardwareInterface</plugin>
           <param name="robot_ip">${robot_ip}</param>
+          <xacro:if value="${gripper == 'ag95'}">
+            <!-- Naming this joint is what switches the hardware's gripper
+                 support on. Everything else comes from fr5.config.yaml, which
+                 the driver replays with SetGripperConfig and ActGripper on
+                 activation. gripper_joint_at_open is the exception: it must
+                 equal the prismatic limit fr5_macro.xacro declares, so it is a
+                 property of the description rather than of the connection. -->
+            <param name="gripper_joint">${prefix}gripper_finger_joint</param>
+            <param name="gripper_joint_at_open">0.0475</param>
+            <param name="gripper_company">${gripper_company}</param>
+            <param name="gripper_device">${gripper_device}</param>
+            <param name="gripper_softversion">${gripper_softversion}</param>
+            <param name="gripper_bus">${gripper_bus}</param>
+            <param name="gripper_index">${gripper_index}</param>
+            <param name="gripper_speed_percent">${gripper_speed_percent}</param>
+            <param name="gripper_force_percent">${gripper_force_percent}</param>
+            <param name="gripper_percent_at_closed">${gripper_percent_at_closed}</param>
+            <param name="gripper_percent_at_open">${gripper_percent_at_open}</param>
+            <!-- Spelled out rather than interpolated: xacro evaluates ${...} as a
+                 Python expression, so a boolean would land in the URDF as
+                 "True"/"False" instead of the canonical lowercase. -->
+            <xacro:if value="${gripper_open_on_activate}">
+              <param name="gripper_open_on_activate">true</param>
+            </xacro:if>
+            <xacro:unless value="${gripper_open_on_activate}">
+              <param name="gripper_open_on_activate">false</param>
+            </xacro:unless>
+            <xacro:if value="${gripper_apply_config}">
+              <param name="gripper_apply_config">true</param>
+            </xacro:if>
+            <xacro:unless value="${gripper_apply_config}">
+              <param name="gripper_apply_config">false</param>
+            </xacro:unless>
+            <xacro:if value="${gripper_required}">
+              <param name="gripper_required">true</param>
+            </xacro:if>
+            <xacro:unless value="${gripper_required}">
+              <param name="gripper_required">false</param>
+            </xacro:unless>
+          </xacro:if>
         </xacro:if>
       </hardware>
@@ -70,4 +138,8 @@
       <xacro:fr5_joint joint_name="${prefix}j5" init="${initial_positions['j5']}" hardware="${hardware}"/>
       <xacro:fr5_joint joint_name="${prefix}j6" init="${initial_positions['j6']}" hardware="${hardware}"/>
+      <xacro:if value="${gripper == 'ag95' and hardware in ('fairino', 'mujoco')}">
+        <xacro:fr5_gripper_joint joint_name="${prefix}gripper_finger_joint"
+                                 with_velocity="${hardware == 'mujoco'}"/>
+      </xacro:if>
     </ros2_control>
   </xacro:macro>

File: cho_description/cho_description_fr5/urdf/fr5.urdf.xacro (robot description, xacro)
@@ -16,4 +16,23 @@
              default="$(find cho_description_fr5)/config/initial_positions.yaml"/>
   <xacro:arg name="mujoco_initial_keyframe" default=""/>
+  <!-- none | ag95. The AG-95 is driven by the robot controller over RS485, so
+       it is only commandable on the real (fairino) build. -->
+  <xacro:arg name="gripper" default="none"/>
+  <!-- RS485 gripper registration, forwarded to the hardware component so it can
+       call SetGripperConfig/ActGripper. The real bringup fills these from
+       cho_bringup_fr5/config/real/fr5.config.yaml; the defaults describe the
+       DAHUAN gripper registered as PGI-140 on end-effector port 1. -->
+  <xacro:arg name="gripper_company" default="4"/>
+  <xacro:arg name="gripper_device" default="0"/>
+  <xacro:arg name="gripper_softversion" default="0"/>
+  <xacro:arg name="gripper_bus" default="1"/>
+  <xacro:arg name="gripper_index" default="1"/>
+  <xacro:arg name="gripper_speed_percent" default="30"/>
+  <xacro:arg name="gripper_force_percent" default="30"/>
+  <xacro:arg name="gripper_percent_at_closed" default="0"/>
+  <xacro:arg name="gripper_percent_at_open" default="100"/>
+  <xacro:arg name="gripper_open_on_activate" default="false"/>
+  <xacro:arg name="gripper_apply_config" default="false"/>
+  <xacro:arg name="gripper_required" default="false"/>
   <xacro:property name="initial_positions_file" default="$(arg initial_positions_file)"/>
   <xacro:property name="initial_positions" value="${xacro.load_yaml(initial_positions_file)}"/>
@@ -24,4 +43,7 @@
     <origin xyz="0 0 0" rpy="0 0 0"/>
   </xacro:fr5_robot>
+  <xacro:if value="${'$(arg gripper)' == 'ag95'}">
+    <xacro:fr5_ag95_gripper prefix="$(arg prefix)" parent="$(arg prefix)tool_tcp"/>
+  </xacro:if>
   <xacro:fr5_ros2_control
     name="fr5_system"
@@ -30,4 +52,17 @@
     robot_ip="$(arg robot_ip)"
     initial_positions="${initial_positions}"
+    gripper="$(arg gripper)"
+    gripper_company="$(arg gripper_company)"
+    gripper_device="$(arg gripper_device)"
+    gripper_softversion="$(arg gripper_softversion)"
+    gripper_bus="$(arg gripper_bus)"
+    gripper_index="$(arg gripper_index)"
+    gripper_speed_percent="$(arg gripper_speed_percent)"
+    gripper_force_percent="$(arg gripper_force_percent)"
+    gripper_percent_at_closed="$(arg gripper_percent_at_closed)"
+    gripper_percent_at_open="$(arg gripper_percent_at_open)"
+    gripper_open_on_activate="$(arg gripper_open_on_activate)"
+    gripper_apply_config="$(arg gripper_apply_config)"
+    gripper_required="$(arg gripper_required)"
     mujoco_initial_keyframe="$(arg mujoco_initial_keyframe)"/>
   <!-- Gazebo (Ignition) ros2_control system plugin. -->

File: cho_description/cho_description_fr5/urdf/fr5_macro.xacro (robot description, xacro)
@@ -233,3 +233,128 @@
     </joint>
   </xacro:macro>
+  <!--
+    DH Robotics AG-95 parallel gripper, bolted straight to the tool flange.
+    `parent` is tool_tcp, which IS the flange face: the wrist3_link collision
+    mesh runs to z = +0.099, so the 100 mm tool_tcp offset is the length of the
+    wrist, not a TCP hanging in free space.
+    The gripper reaches 200.8 mm past that face and is 168 mm across, and until
+    it was modelled MoveIt planned as though that volume were empty - which is
+    what drove the gripper into the arm. Geometry now comes from the vendored
+    upstream meshes; see the macro below and meshes/ag95/README.md.
+    Both jaws move symmetrically, so one finger travels half the stroke. The
+    single finger joint stands for that half; cho_controller_gripper maps it back
+    to the full opening through width_at_open.
+  -->
+  <xacro:macro name="fr5_ag95_gripper" params="prefix parent yaw:=0">
+    <!--
+      One link carries the whole gripper: three collision elements on
+      gripper_base_link rather than a link per part, because every extra link is
+      another row in MoveIt's collision matrix and another SRDF pair to reason
+      about, for no gain when the parts do not move independently.
+      The two meshes are the AG-95 parts that are RIGID with respect to the
+      flange, taken unmodified from the vendored upstream model (millimetres,
+      hence the scale) and placed at the origin, which is where upstream's own
+      base and body transforms compose to. The box covers the jaws: their swept
+      volume over the entire 0-to-closed stroke, measured off the same meshes
+      (see meshes/ag95/README.md). Conservative on purpose - a fixed box that
+      encloses every jaw position can refuse a plan the real gripper would have
+      cleared, but it can never pass one the real gripper would have hit.
+      `yaw` is the rotation about the flange axis, and 0 is confirmed correct for
+      this cell rather than assumed: the operator's own fr5_ag95 URDF mounts the
+      gripper on a `tool0` whose net transform from wrist3_link is
+      xyz (0, 0, 0.1) with an IDENTITY rotation - the same frame as tool_tcp
+      here - and places the two jaw knuckles at x = -0.016 and +0.016 in it, so
+      the jaws separate along x, which is the finger axis below. Keep the
+      parameter anyway: bolting the gripper on a quarter turn round would
+      otherwise silently rotate a 168 x 51 mm box by 90 degrees.
+      Mass is the upstream figure, independently corroborated by the operator's
+      own URDF at 0.83416 kg, and is carried for completeness only: the FR5 is
+      position-controlled and the robot controller does its own gravity
+      compensation, so the payload that matters is the one set on the teach
+      pendant, not this number.
+      On gripper length the two available models disagree - the operator's URDF
+      puts its grasp frame at z = 170 mm and the vendored upstream one at
+      190 mm - which is exactly why the jaw box is sized from the swept mesh
+      envelope (200.8 mm) rather than from either grasp frame: it encloses both.
+    -->
+    <link name="${prefix}gripper_base_link">
+      <inertial>
+        <origin xyz="0 0 0.0655" rpy="0 0 0"/>
+        <mass value="0.8347"/>
+        <inertia ixx="0.0025" ixy="0.0" ixz="0.0" iyy="0.0025" iyz="0.0" izz="0.0008"/>
+      </inertial>
+      <visual>
+        <origin xyz="0 0 0" rpy="0 0 0"/>
+        <geometry>
+          <mesh filename="package://cho_description_fr5/meshes/ag95/visual/base_link.stl"
+                scale="0.001 0.001 0.001"/>
+        </geometry>
+        <material name="fr5_ag95_plate">
+          <color rgba="0.79216 0.81961 0.93333 1"/>
+        </material>
+      </visual>
+      <visual>
+        <origin xyz="0 0 0" rpy="0 0 0"/>
+        <geometry>
+          <mesh filename="package://cho_description_fr5/meshes/ag95/visual/gripper_body.stl"
+                scale="0.001 0.001 0.001"/>
+        </geometry>
+        <material name="fr5_ag95_body">
+          <color rgba="0.15 0.15 0.15 1"/>
+        </material>
+      </visual>
+      <collision>
+        <origin xyz="0 0 0" rpy="0 0 0"/>
+        <geometry>
+          <mesh filename="package://cho_description_fr5/meshes/ag95/collision/base_link.stl"
+                scale="0.001 0.001 0.001"/>
+        </geometry>
+      </collision>
+      <collision>
+        <origin xyz="0 0 0" rpy="0 0 0"/>
+        <geometry>
+          <mesh filename="package://cho_description_fr5/meshes/ag95/collision/gripper_body.stl"
+                scale="0.001 0.001 0.001"/>
+        </geometry>
+      </collision>
+      <!-- The jaw envelope is drawn as well as checked, translucent so it reads
+           as a swept volume rather than as fingers. Seeing exactly what the
+           planner collides against beats seeing prettier geometry that does
+           not match it. -->
+      <visual>
+        <origin xyz="0 0 0.1456" rpy="0 0 0"/>
+        <geometry>
+          <box size="0.1682 0.0508 0.1104"/>
+        </geometry>
+        <material name="fr5_ag95_jaw_envelope">
+          <color rgba="0.9 0.6 0.2 0.25"/>
+        </material>
+      </visual>
+      <collision>
+        <!-- Jaw sweep: x 168.2, y 50.8, z 90.4 to 200.8 mm from the flange. -->
+        <origin xyz="0 0 0.1456" rpy="0 0 0"/>
+        <geometry>
+          <box size="0.1682 0.0508 0.1104"/>
+        </geometry>
+      </collision>
+    </link>
+    <joint name="${prefix}flange_to_gripper" type="fixed">
+      <parent link="${parent}"/>
+      <child link="${prefix}gripper_base_link"/>
+      <origin xyz="0 0 0" rpy="0 0 ${yaw}"/>
+    </joint>
+    <!-- The commanded finger. Geometry-free: the jaws are already covered by the
+         box above, and giving this link its own body would double-count them.
+         Axis x, matching the direction the upstream linkage actually drives the
+         jaws. Both jaws move, so this one joint stands for half the stroke. -->
+    <link name="${prefix}gripper_finger_link"/>
+    <joint name="${prefix}gripper_finger_joint" type="prismatic">
+      <parent link="${prefix}gripper_base_link"/>
+      <child link="${prefix}gripper_finger_link"/>
+      <origin xyz="0 0 0.1456" rpy="0 0 0"/>
+      <axis xyz="1 0 0"/>
+      <!-- Half of the 95 mm stroke: 0 closed, 0.0475 fully open. -->
+      <limit lower="0.0" upper="0.0475" effort="100.0" velocity="0.15"/>
+    </joint>
+  </xacro:macro>
 </robot>
