Commit message: Add fail-closed OpenArm MIT real bringup

File: cho_description/cho_description_openarm/robots/openarm_v10/openarm_v10.ros2_control.xacro (robot description, xacro)
@@ -28,4 +28,10 @@
       mujoco_mit_prototype:=false
       mujoco_mit_headless:=false
+      real_mit_hardware:=false
+      real_mit_safety_profile:=real_conservative_unapproved
+      mit_expected_update_rate_hz:=200
+      open_can:=false
+      enable_motors:=false
+      operator_approval:=false
       bimanual:=false
       arm_prefix:=''
@@ -42,5 +48,8 @@
       runtime_param_file:=''
       description_pkg:=cho_description_openarm">
-    <xacro:property name="mit_gains" value="${hardware == 'real' or hardware == 'mock'}"/>
+    <!-- The legacy upstream real/mock component exports position, velocity and
+         effort only. The Cho MIT real adapter has the same five-tuple contract
+         as the MuJoCo adapter, so keep that path separate. -->
+    <xacro:property name="mit_gains" value="${hardware == 'mock' or (hardware == 'real' and not real_mit_hardware)}"/>
     <xacro:property name="scene_dir" value="${'openarm_v10_bimanual' if bimanual else 'openarm_v10'}"/>
     <!--
@@ -98,4 +107,28 @@
           <param name="kd_hand">${control_gains['hand']['kd']}</param>
     </xacro:macro>
+    <!--
+      Real MIT transport contract.  All three permission values default to
+      false in the description as well as in the launch file: rendering a
+      real URDF or starting robot_state_publisher must never open a CAN socket
+      or enable a motor.  The adapter validates the conjunction of open_can
+      and operator_approval before constructing its vendor transport, and also
+      keeps motors disabled unless enable_motors is explicitly true.
+      The default safety profile is intentionally unapproved.  The launch
+      permits the separate commissioning profile only after all three runtime
+      acknowledgement flags are true; the adapter checks that profile again
+      before transport construction.
+    -->
+    <xacro:macro name="openarm_mit_real_hw_params" params="side can">
+      <plugin>cho_hardware_openarm_mit_real/OpenArmMitRealSystem</plugin>
+      <param name="mit_safety_profile_file">$(find cho_description_openarm)/config/mit_safety_profiles_v1.yaml</param>
+      <param name="mit_safety_profile">${real_mit_safety_profile}</param>
+      <param name="mit_expected_update_rate_hz">${mit_expected_update_rate_hz}</param>
+      <param name="can_interface">${can}</param>
+      <param name="can_fd">${can_fd}</param>
+      <param name="arm_side">${side}</param>
+      <param name="open_can">${open_can}</param>
+      <param name="enable_motors">${enable_motors}</param>
+      <param name="operator_approval">${operator_approval}</param>
+    </xacro:macro>
     <xacro:macro name="configure_joint" params="joint_name initial_position:=0.0 gripper:=false">
       <joint name="${joint_name}">
@@ -106,5 +139,5 @@
         </xacro:if>
         <xacro:unless value="${mit_gains}">
-          <xacro:if value="${hardware == 'mujoco' and mujoco_mit_prototype}">
+          <xacro:if value="${(hardware == 'mujoco' and mujoco_mit_prototype) or (hardware == 'real' and real_mit_hardware)}">
             <xacro:if value="${gripper}"><command_interface name="position"/></xacro:if>
             <xacro:unless value="${gripper}"><command_interface name="position"/><command_interface name="velocity"/><command_interface name="stiffness"/><command_interface name="damping"/><command_interface name="effort"/></xacro:unless>
@@ -154,9 +187,30 @@
     </xacro:macro>
     <!-- Only finger_joint1 is actuated. finger_joint2 is a URDF <mimic> of it
-         (and a MuJoCo equality constraint), so it carries no interfaces. -->
+         (and a MuJoCo equality constraint), so it carries no interfaces. The
+         new real MIT adapter intentionally owns exactly seven arm motors; it
+         has no gripper transport yet, therefore real_mit_hardware never adds
+         a finger interface to that SystemInterface. The hand geometry remains
+         in the URDF for visualization. -->
     <xacro:macro name="one_hand_joints" params="prefix">
-      <xacro:if value="${hand}">
+      <xacro:if value="${hand and not (hardware == 'real' and real_mit_hardware)}">
         <xacro:configure_joint joint_name="openarm_${prefix}finger_joint1" gripper="true"/>
       </xacro:if>
+    </xacro:macro>
+    <!-- The direct MIT controller claims these four command and five state
+         GPIO interfaces together with all five fields of every arm joint. A
+         real bimanual build has two SystemInterfaces, so each component owns
+         only its own arm-scoped GPIO resource. -->
+    <xacro:macro name="mit_arm_gpio" params="resource">
+      <gpio name="${resource}">
+        <command_interface name="mit_session_echo"/>
+        <command_interface name="mit_lease_cycles"/>
+        <command_interface name="mit_commit_generation"/>
+        <command_interface name="mit_safe_request_generation"/>
+        <state_interface name="mit_session_id"/>
+        <state_interface name="mit_ack_generation"/>
+        <state_interface name="mit_safe_generation"/>
+        <state_interface name="mit_safe_ack_generation"/>
+        <state_interface name="mit_status"/>
+      </gpio>
     </xacro:macro>
     <!-- The bimanual build is one model with two chains, so both arms' joints go
@@ -222,15 +276,31 @@
       <ros2_control name="OpenArmLeftHardwareInterface" type="system">
         <hardware>
-          <xacro:openarm_hw_params prefix="left_" can="${left_can_interface}"/>
+          <xacro:if value="${real_mit_hardware}">
+            <xacro:openarm_mit_real_hw_params side="left" can="${left_can_interface}"/>
+          </xacro:if>
+          <xacro:unless value="${real_mit_hardware}">
+            <xacro:openarm_hw_params prefix="left_" can="${left_can_interface}"/>
+          </xacro:unless>
         </hardware>
         <xacro:one_arm_joints prefix="left_"/>
         <xacro:one_hand_joints prefix="left_"/>
+        <xacro:if value="${real_mit_hardware}">
+          <xacro:mit_arm_gpio resource="openarm_left_arm"/>
+        </xacro:if>
       </ros2_control>
       <ros2_control name="OpenArmRightHardwareInterface" type="system">
         <hardware>
-          <xacro:openarm_hw_params prefix="right_" can="${right_can_interface}"/>
+          <xacro:if value="${real_mit_hardware}">
+            <xacro:openarm_mit_real_hw_params side="right" can="${right_can_interface}"/>
+          </xacro:if>
+          <xacro:unless value="${real_mit_hardware}">
+            <xacro:openarm_hw_params prefix="right_" can="${right_can_interface}"/>
+          </xacro:unless>
         </hardware>
         <xacro:one_arm_joints prefix="right_"/>
         <xacro:one_hand_joints prefix="right_"/>
+        <xacro:if value="${real_mit_hardware}">
+          <xacro:mit_arm_gpio resource="openarm_right_arm"/>
+        </xacro:if>
       </ros2_control>
     </xacro:if>
@@ -240,5 +310,10 @@
         <hardware>
           <xacro:if value="${hardware == 'real'}">
-            <xacro:openarm_hw_params prefix="${arm_prefix}" can="${can_interface}"/>
+            <xacro:if value="${real_mit_hardware}">
+              <xacro:openarm_mit_real_hw_params side="single" can="${can_interface}"/>
+            </xacro:if>
+            <xacro:unless value="${real_mit_hardware}">
+              <xacro:openarm_hw_params prefix="${arm_prefix}" can="${can_interface}"/>
+            </xacro:unless>
           </xacro:if>
           <xacro:if value="${hardware == 'mock'}">
@@ -282,5 +357,5 @@
         <xacro:arm_joints/>
         <xacro:hand_joints/>
-        <xacro:if value="${hardware == 'mujoco' and mujoco_mit_prototype}">
+        <xacro:if value="${(hardware == 'mujoco' and mujoco_mit_prototype) or (hardware == 'real' and real_mit_hardware)}">
           <xacro:if value="${bimanual}">
             <gpio name="openarm_left_arm"><command_interface name="mit_session_echo"/><command_interface name="mit_lease_cycles"/><command_interface name="mit_commit_generation"/><command_interface name="mit_safe_request_generation"/><state_interface name="mit_session_id"/><state_interface name="mit_ack_generation"/><state_interface name="mit_safe_generation"/><state_interface name="mit_safe_ack_generation"/><state_interface name="mit_status"/></gpio>

File: cho_description/cho_description_openarm/robots/openarm_v10/openarm_v10.urdf.xacro (robot description, xacro)
@@ -35,4 +35,12 @@
   <xacro:arg name="mujoco_mit_prototype" default="false"/>
   <xacro:arg name="mujoco_mit_headless" default="false"/>
+  <!-- Real MIT transport is explicit and fail-closed.  These values are
+       forwarded only to the Cho real adapter; all defaults are non-driving. -->
+  <xacro:arg name="real_mit_hardware" default="false"/>
+  <xacro:arg name="real_mit_safety_profile" default="real_conservative_unapproved"/>
+  <xacro:arg name="mit_expected_update_rate_hz" default="200"/>
+  <xacro:arg name="open_can" default="false"/>
+  <xacro:arg name="enable_motors" default="false"/>
+  <xacro:arg name="operator_approval" default="false"/>
   <xacro:arg name="bimanual"      default="false"/>
   <xacro:arg name="arm_prefix"    default=""/>
@@ -131,4 +139,10 @@
       mujoco_mit_prototype="$(arg mujoco_mit_prototype)"
       mujoco_mit_headless="$(arg mujoco_mit_headless)"
+      real_mit_hardware="$(arg real_mit_hardware)"
+      real_mit_safety_profile="$(arg real_mit_safety_profile)"
+      mit_expected_update_rate_hz="$(arg mit_expected_update_rate_hz)"
+      open_can="$(arg open_can)"
+      enable_motors="$(arg enable_motors)"
+      operator_approval="$(arg operator_approval)"
       bimanual="$(arg bimanual)"
       arm_prefix="$(arg arm_prefix)"

Commit message: Run the real OpenArm MIT bus at 750 Hz with state from the command reply
Safety profile: 750 Hz commissioning envelope with the lease, refresh and
stale-state cycle counts rescaled to keep the 50/100 ms wall-clock timeouts,
canonical OpenArm position/velocity limits, manufacturer peak torques
(40/40/27/27/7/7/7) instead of the packet encoding range, task gain ceilings
sized for zeta 0.7 through the drive with kd capped at 5, separate
return-to-zero ceilings and tau_ff slews the gravity term can follow.

Real adapter: optional state from the reply the MIT command frame already
produces, so the redundant 0xCC query is gone and 7 tx + 7 rx per cycle fits
in half the CAN FD bus. Every tuple is validated per joint against the
profile before it reaches the bus. Per-joint safe-hold gains.

Description: the same limits in joint_limits.yaml, the ros2_control block
forwards the new adapter parameters, plus an rviz config for the bringup.

File: cho_description/cho_description_openarm/robots/openarm_v10/openarm_v10.ros2_control.xacro (robot description, xacro)
@@ -29,9 +29,7 @@
       mujoco_mit_headless:=false
       real_mit_hardware:=false
-      real_mit_safety_profile:=real_conservative_unapproved
+      real_mit_arm:=both_independent
+      real_mit_safety_profile:=real_conservative_commissioning
       mit_expected_update_rate_hz:=200
-      open_can:=false
-      enable_motors:=false
-      operator_approval:=false
       bimanual:=false
       arm_prefix:=''
@@ -41,4 +39,5 @@
       right_can_interface:=can0
       can_fd:=true
+      mit_state_from_command_reply:=false
       ee_type:=parallel_link
       kp_scale:=0.0
@@ -74,4 +73,5 @@
           <param name="can_interface">${can}</param>
           <param name="can_fd">${can_fd}</param>
+          <param name="mit_state_from_command_reply">${mit_state_from_command_reply}</param>
           <param name="hand">${hand}</param>
           <param name="ee_type">${ee_type}</param>
@@ -108,14 +108,7 @@
     </xacro:macro>
     <!--
-      Real MIT transport contract.  All three permission values default to
-      false in the description as well as in the launch file: rendering a
-      real URDF or starting robot_state_publisher must never open a CAN socket
-      or enable a motor.  The adapter validates the conjunction of open_can
-      and operator_approval before constructing its vendor transport, and also
-      keeps motors disabled unless enable_motors is explicitly true.
-      The default safety profile is intentionally unapproved.  The launch
-      permits the separate commissioning profile only after all three runtime
-      acknowledgement flags are true; the adapter checks that profile again
-      before transport construction.
+      Real MIT transport contract. The launch selects an explicit real
+      commissioning profile; the adapter validates that profile and the CAN
+      interface before constructing its vendor transport.
     -->
     <xacro:macro name="openarm_mit_real_hw_params" params="side can">
@@ -126,8 +119,6 @@
       <param name="can_interface">${can}</param>
       <param name="can_fd">${can_fd}</param>
+          <param name="mit_state_from_command_reply">${mit_state_from_command_reply}</param>
       <param name="arm_side">${side}</param>
-      <param name="open_can">${open_can}</param>
-      <param name="enable_motors">${enable_motors}</param>
-      <param name="operator_approval">${operator_approval}</param>
     </xacro:macro>
     <xacro:macro name="configure_joint" params="joint_name initial_position:=0.0 gripper:=false">
@@ -143,5 +134,5 @@
             <xacro:unless value="${gripper}"><command_interface name="position"/><command_interface name="velocity"/><command_interface name="stiffness"/><command_interface name="damping"/><command_interface name="effort"/></xacro:unless>
           </xacro:if>
-          <xacro:unless value="${hardware == 'mujoco' and mujoco_mit_prototype}">
+          <xacro:unless value="${(hardware == 'mujoco' and mujoco_mit_prototype) or (hardware == 'real' and real_mit_hardware)}">
           <!-- The gripper is position-driven in every simulator actuator set
                (its MJCF actuator is a position servo on the "split" tendon in
@@ -185,4 +176,17 @@
       <xacro:configure_joint joint_name="openarm_${prefix}joint6"/>
       <xacro:configure_joint joint_name="openarm_${prefix}joint7"/>
+    </xacro:macro>
+    <!-- A non-selected real bimanual arm exists for visualization only.  It
+         intentionally exports state interfaces and no command interfaces, so
+         GenericSystem keeps these URDF initial values frozen and no controller
+         can claim the visualization-only arm. -->
+    <xacro:macro name="one_arm_visualization_joints" params="prefix">
+      <joint name="openarm_${prefix}joint1"><state_interface name="position"><param name="initial_value">0.0</param></state_interface><state_interface name="velocity"/><state_interface name="effort"/></joint>
+      <joint name="openarm_${prefix}joint2"><state_interface name="position"><param name="initial_value">0.0</param></state_interface><state_interface name="velocity"/><state_interface name="effort"/></joint>
+      <joint name="openarm_${prefix}joint3"><state_interface name="position"><param name="initial_value">0.0</param></state_interface><state_interface name="velocity"/><state_interface name="effort"/></joint>
+      <joint name="openarm_${prefix}joint4"><state_interface name="position"><param name="initial_value">0.3</param></state_interface><state_interface name="velocity"/><state_interface name="effort"/></joint>
+      <joint name="openarm_${prefix}joint5"><state_interface name="position"><param name="initial_value">0.0</param></state_interface><state_interface name="velocity"/><state_interface name="effort"/></joint>
+      <joint name="openarm_${prefix}joint6"><state_interface name="position"><param name="initial_value">0.0</param></state_interface><state_interface name="velocity"/><state_interface name="effort"/></joint>
+      <joint name="openarm_${prefix}joint7"><state_interface name="position"><param name="initial_value">0.0</param></state_interface><state_interface name="velocity"/><state_interface name="effort"/></joint>
     </xacro:macro>
     <!-- Only finger_joint1 is actuated. finger_joint2 is a URDF <mimic> of it
@@ -274,8 +278,13 @@
          talking to its own socket. -->
     <xacro:if value="${hardware == 'real' and bimanual}">
+      <xacro:property name="left_real_mit_selected" value="${real_mit_arm == 'left' or real_mit_arm == 'both_independent'}"/>
+      <xacro:property name="right_real_mit_selected" value="${real_mit_arm == 'right' or real_mit_arm == 'both_independent'}"/>
       <ros2_control name="OpenArmLeftHardwareInterface" type="system">
         <hardware>
-          <xacro:if value="${real_mit_hardware}">
+          <xacro:if value="${real_mit_hardware and left_real_mit_selected}">
             <xacro:openarm_mit_real_hw_params side="left" can="${left_can_interface}"/>
+          </xacro:if>
+          <xacro:if value="${real_mit_hardware and not left_real_mit_selected}">
+            <plugin>mock_components/GenericSystem</plugin>
           </xacro:if>
           <xacro:unless value="${real_mit_hardware}">
@@ -283,7 +292,8 @@
           </xacro:unless>
         </hardware>
-        <xacro:one_arm_joints prefix="left_"/>
+        <xacro:if value="${not real_mit_hardware or left_real_mit_selected}"><xacro:one_arm_joints prefix="left_"/></xacro:if>
+        <xacro:if value="${real_mit_hardware and not left_real_mit_selected}"><xacro:one_arm_visualization_joints prefix="left_"/></xacro:if>
         <xacro:one_hand_joints prefix="left_"/>
-        <xacro:if value="${real_mit_hardware}">
+        <xacro:if value="${real_mit_hardware and left_real_mit_selected}">
           <xacro:mit_arm_gpio resource="openarm_left_arm"/>
         </xacro:if>
@@ -291,6 +301,9 @@
       <ros2_control name="OpenArmRightHardwareInterface" type="system">
         <hardware>
-          <xacro:if value="${real_mit_hardware}">
+          <xacro:if value="${real_mit_hardware and right_real_mit_selected}">
             <xacro:openarm_mit_real_hw_params side="right" can="${right_can_interface}"/>
+          </xacro:if>
+          <xacro:if value="${real_mit_hardware and not right_real_mit_selected}">
+            <plugin>mock_components/GenericSystem</plugin>
           </xacro:if>
           <xacro:unless value="${real_mit_hardware}">
@@ -298,7 +311,8 @@
           </xacro:unless>
         </hardware>
-        <xacro:one_arm_joints prefix="right_"/>
+        <xacro:if value="${not real_mit_hardware or right_real_mit_selected}"><xacro:one_arm_joints prefix="right_"/></xacro:if>
+        <xacro:if value="${real_mit_hardware and not right_real_mit_selected}"><xacro:one_arm_visualization_joints prefix="right_"/></xacro:if>
         <xacro:one_hand_joints prefix="right_"/>
-        <xacro:if value="${real_mit_hardware}">
+        <xacro:if value="${real_mit_hardware and right_real_mit_selected}">
           <xacro:mit_arm_gpio resource="openarm_right_arm"/>
         </xacro:if>

File: cho_description/cho_description_openarm/robots/openarm_v10/openarm_v10.urdf.xacro (robot description, xacro)
@@ -35,12 +35,9 @@
   <xacro:arg name="mujoco_mit_prototype" default="false"/>
   <xacro:arg name="mujoco_mit_headless" default="false"/>
-  <!-- Real MIT transport is explicit and fail-closed.  These values are
-       forwarded only to the Cho real adapter; all defaults are non-driving. -->
+  <!-- Real MIT transport uses an explicit commissioning profile. -->
   <xacro:arg name="real_mit_hardware" default="false"/>
-  <xacro:arg name="real_mit_safety_profile" default="real_conservative_unapproved"/>
+  <xacro:arg name="real_mit_arm" default="both_independent"/>
+  <xacro:arg name="real_mit_safety_profile" default="real_conservative_commissioning"/>
   <xacro:arg name="mit_expected_update_rate_hz" default="200"/>
-  <xacro:arg name="open_can" default="false"/>
-  <xacro:arg name="enable_motors" default="false"/>
-  <xacro:arg name="operator_approval" default="false"/>
   <xacro:arg name="bimanual"      default="false"/>
   <xacro:arg name="arm_prefix"    default=""/>
@@ -62,4 +59,5 @@
   <xacro:arg name="right_arm_base_rpy"  default="1.5708 0 0"/>
   <xacro:arg name="can_fd"        default="true"/>
+  <xacro:arg name="mit_state_from_command_reply" default="false"/>
   <xacro:arg name="kp_scale"      default="0.0"/>
   <xacro:arg name="kd_scale"      default="1.0"/>
@@ -140,9 +138,7 @@
       mujoco_mit_headless="$(arg mujoco_mit_headless)"
       real_mit_hardware="$(arg real_mit_hardware)"
+      real_mit_arm="$(arg real_mit_arm)"
       real_mit_safety_profile="$(arg real_mit_safety_profile)"
       mit_expected_update_rate_hz="$(arg mit_expected_update_rate_hz)"
-      open_can="$(arg open_can)"
-      enable_motors="$(arg enable_motors)"
-      operator_approval="$(arg operator_approval)"
       bimanual="$(arg bimanual)"
       arm_prefix="$(arg arm_prefix)"
@@ -152,4 +148,5 @@
       can_interface="$(arg can_interface)"
       can_fd="$(arg can_fd)"
+      mit_state_from_command_reply="$(arg mit_state_from_command_reply)"
       ee_type="parallel_link"
       kp_scale="$(arg kp_scale)"
