Commit message: Give the real OpenArm adapter the hand on its own CAN contract
With hand:=true the adapter owns an eighth Damiao motor on the same socket as
the seven arm motors and exports the finger as an ordinary position +
max_effort joint. It stays outside the MIT arm contract exactly as
docs/openarm_mit_contract_v1.md requires: no arm vector, lease generation or
SAFE acknowledgement carries a gripper value, and the gripper controller
cannot claim an MIT tuple field. Only failure couples back, and then the arm
is safed, because the two share a bus.

POS_FORCE rather than an MIT tuple, so the drive caps its own current and the
action's force field is a real limit; the legacy MIT path stays available for
firmware where that mode is not live. Writes are decimated to a fifth of the
control rate: the finger has no dynamics worth 750 Hz and every frame it sends
is one the arm cannot use.

The joint-to-motor map is configured at both ends because the motor zero is
wherever the hand was last zeroed and it opens in the negative direction.
Activation seeds the command from the measured finger, since ros2_control
initialises a command interface to zero and zero on this map is fully closed -
an unseeded command would slam the hand shut on whatever it was holding.

Measured on the right hand 2026-09-05: action moves to 40, 70 and 88 mm all
landed within 80 um, and a continuous width command tracked to 30 um.

File: cho_description/cho_description_openarm/robots/openarm_v10/openarm_v10.ros2_control.xacro (robot description, xacro)
@@ -40,4 +40,14 @@
       can_fd:=true
       mit_state_from_command_reply:=false
+      gripper_send_can_id:=8
+      gripper_recv_can_id:=24
+      gripper_pos_force:=true
+      gripper_speed_rad_s:=5.0
+      gripper_joint_closed:=0.0
+      gripper_joint_open:=0.044
+      gripper_motor_closed:=0.0
+      gripper_motor_open:=-1.0472
+      gripper_max_force:=9.0
+      gripper_write_decimation:=5
       ee_type:=parallel_link
       kp_scale:=0.0
@@ -121,4 +131,24 @@
           <param name="mit_state_from_command_reply">${mit_state_from_command_reply}</param>
       <param name="arm_side">${side}</param>
+      <!-- The gripper is one more Damiao motor on this same CAN socket, but
+           outside the MIT arm contract: its values never enter an arm vector,
+           a lease generation or a SAFE acknowledgement. Only its failure
+           couples back, and then the arm is safed because they share a bus.
+           The motor endpoints are measured on the physical hand: the motor
+           zero is wherever it was last zeroed and it opens in the negative
+           direction, so both ends are configured rather than assumed. -->
+      <param name="hand">${hand}</param>
+      <xacro:if value="${hand}">
+        <param name="gripper_send_can_id">${gripper_send_can_id}</param>
+        <param name="gripper_recv_can_id">${gripper_recv_can_id}</param>
+        <param name="gripper_pos_force">${gripper_pos_force}</param>
+        <param name="gripper_speed_rad_s">${gripper_speed_rad_s}</param>
+        <param name="gripper_joint_closed">${gripper_joint_closed}</param>
+        <param name="gripper_joint_open">${gripper_joint_open}</param>
+        <param name="gripper_motor_closed">${gripper_motor_closed}</param>
+        <param name="gripper_motor_open">${gripper_motor_open}</param>
+        <param name="gripper_max_force">${gripper_max_force}</param>
+        <param name="gripper_write_decimation">${gripper_write_decimation}</param>
+      </xacro:if>
     </xacro:macro>
     <xacro:macro name="configure_joint" params="joint_name initial_position:=0.0 gripper:=false">
@@ -131,5 +161,12 @@
         <xacro:unless value="${mit_gains}">
           <xacro:if value="${(hardware == 'mujoco' and mujoco_mit_prototype) or (hardware == 'real' and real_mit_hardware)}">
-            <xacro:if value="${gripper}"><command_interface name="position"/></xacro:if>
+            <!-- max_effort is the grasp force in newtons at the finger; the
+                 adapter scales it into the drive's per-unit current cap. Only
+                 the real adapter exports it - MuJoCo's finger is a position
+                 servo on a tendon and would reject the extra interface. -->
+            <xacro:if value="${gripper}">
+              <command_interface name="position"/>
+              <xacro:if value="${hardware == 'real'}"><command_interface name="max_effort"/></xacro:if>
+            </xacro:if>
             <xacro:unless value="${gripper}"><command_interface name="position"/><command_interface name="velocity"/><command_interface name="stiffness"/><command_interface name="damping"/><command_interface name="effort"/></xacro:unless>
           </xacro:if>
@@ -196,7 +233,19 @@
          a finger interface to that SystemInterface. The hand geometry remains
          in the URDF for visualization. -->
-    <xacro:macro name="one_hand_joints" params="prefix">
-      <xacro:if value="${hand and not (hardware == 'real' and real_mit_hardware)}">
-        <xacro:configure_joint joint_name="openarm_${prefix}finger_joint1" gripper="true"/>
+    <xacro:macro name="one_hand_joints" params="prefix mit_selected:=true">
+      <xacro:if value="${hand}">
+        <!-- A real bimanual arm this bringup did not select is a state-only
+             GenericSystem for visualization, so its finger must not export a
+             command interface either - nothing exists to drive it. -->
+        <xacro:if value="${hardware == 'real' and real_mit_hardware and not mit_selected}">
+          <joint name="openarm_${prefix}finger_joint1">
+            <state_interface name="position"><param name="initial_value">0.0</param></state_interface>
+            <state_interface name="velocity"/>
+            <state_interface name="effort"/>
+          </joint>
+        </xacro:if>
+        <xacro:unless value="${hardware == 'real' and real_mit_hardware and not mit_selected}">
+          <xacro:configure_joint joint_name="openarm_${prefix}finger_joint1" gripper="true"/>
+        </xacro:unless>
       </xacro:if>
     </xacro:macro>
@@ -294,5 +343,5 @@
         <xacro:if value="${not real_mit_hardware or left_real_mit_selected}"><xacro:one_arm_joints prefix="left_"/></xacro:if>
         <xacro:if value="${real_mit_hardware and not left_real_mit_selected}"><xacro:one_arm_visualization_joints prefix="left_"/></xacro:if>
-        <xacro:one_hand_joints prefix="left_"/>
+        <xacro:one_hand_joints prefix="left_" mit_selected="${left_real_mit_selected}"/>
         <xacro:if value="${real_mit_hardware and left_real_mit_selected}">
           <xacro:mit_arm_gpio resource="openarm_left_arm"/>
@@ -313,5 +362,5 @@
         <xacro:if value="${not real_mit_hardware or right_real_mit_selected}"><xacro:one_arm_joints prefix="right_"/></xacro:if>
         <xacro:if value="${real_mit_hardware and not right_real_mit_selected}"><xacro:one_arm_visualization_joints prefix="right_"/></xacro:if>
-        <xacro:one_hand_joints prefix="right_"/>
+        <xacro:one_hand_joints prefix="right_" mit_selected="${right_real_mit_selected}"/>
         <xacro:if value="${real_mit_hardware and right_real_mit_selected}">
           <xacro:mit_arm_gpio resource="openarm_right_arm"/>

File: cho_description/cho_description_openarm/robots/openarm_v10/openarm_v10.urdf.xacro (robot description, xacro)
@@ -60,4 +60,18 @@
   <xacro:arg name="can_fd"        default="true"/>
   <xacro:arg name="mit_state_from_command_reply" default="false"/>
+  <!-- Real gripper. The CAN ids are upstream OpenArm's defaults (0x08 / 0x18)
+       expressed in decimal because xacro parses these as numbers. The motor
+       endpoints are measured on the physical hand: zero is wherever it was last
+       zeroed and it opens negative. -->
+  <xacro:arg name="gripper_send_can_id" default="8"/>
+  <xacro:arg name="gripper_recv_can_id" default="24"/>
+  <xacro:arg name="gripper_pos_force" default="true"/>
+  <xacro:arg name="gripper_speed_rad_s" default="5.0"/>
+  <xacro:arg name="gripper_joint_closed" default="0.0"/>
+  <xacro:arg name="gripper_joint_open" default="0.044"/>
+  <xacro:arg name="gripper_motor_closed" default="0.0"/>
+  <xacro:arg name="gripper_motor_open" default="-1.0472"/>
+  <xacro:arg name="gripper_max_force" default="9.0"/>
+  <xacro:arg name="gripper_write_decimation" default="5"/>
   <xacro:arg name="kp_scale"      default="0.0"/>
   <xacro:arg name="kd_scale"      default="1.0"/>
@@ -149,4 +163,14 @@
       can_fd="$(arg can_fd)"
       mit_state_from_command_reply="$(arg mit_state_from_command_reply)"
+      gripper_send_can_id="$(arg gripper_send_can_id)"
+      gripper_recv_can_id="$(arg gripper_recv_can_id)"
+      gripper_pos_force="$(arg gripper_pos_force)"
+      gripper_speed_rad_s="$(arg gripper_speed_rad_s)"
+      gripper_joint_closed="$(arg gripper_joint_closed)"
+      gripper_joint_open="$(arg gripper_joint_open)"
+      gripper_motor_closed="$(arg gripper_motor_closed)"
+      gripper_motor_open="$(arg gripper_motor_open)"
+      gripper_max_force="$(arg gripper_max_force)"
+      gripper_write_decimation="$(arg gripper_write_decimation)"
       ee_type="parallel_link"
       kp_scale="$(arg kp_scale)"
