Commit message: Move the Bota FT sensor and the forge tasks out of the core, keeping the hooks a project mounts its own parts with
The core's Franka FR3 carried a Bota SensONE setup and three FORGE tasks that
only one project, FIRe, uses. They now live in that project's overlay
workspace; the core's robot has no sensor in any bringup, and a project mounts
one through general extension points:

- franka_robot.xacro takes ee_connection_xacro, a xacro file whose
  ee_connection(arm_prefix, robot_type) macro adds parts on fr3_link8, and
  special_connection is again what upstream made it: the link the hand hangs
  off. The real and Gazebo bringups take both.
- Every Franka bringup takes payload_file (empty: config/payload.yaml, the
  hand alone). MuJoCo's xacro_file defaults to urdf/fr3, whose ros2_control
  block names its model; a project robot brings both.
- Isaac's ft_link publishes a link's incoming joint load as a raw Wrench on
  /isaac/ft_raw, replacing publish_ft and the Bota emulation node.
  load_ft_sensor is gone from every bringup.
- SafetyMonitorBehavior's wrench_topic has no default; a force or torque
  limit needs it.

Removed: urdf/ and xml/fr3_with_ft_sensor, the sensor's mounting mesh,
payload_ft_sensor.yaml, cho_sensor/bota_ft_sensor, the bota_driver_ros2 and
bota_driver_ros2_example submodules, isaac_ft_sensor.py, the tasks
peg_insert, gear_mesh and nut_thread with their test, TareFTSensorServiceBehavior
and tare_ft_children.

urdf/fr3 is now the FT URDF without the sensor, so it keeps that file's MuJoCo
and Isaac blocks; MuJoCo's default description drops joint7's unused
safety_controller and dynamics, as the FT URDF never had them. Isaac defaults
to it and to usd/fr3 (built locally, not tracked).

Launch goldens regenerated: mounted (real, Gazebo) and payload (MuJoCo) cases
use stand-ins in launch_golden/fake/, which test_goal_frames reads for <FAKE>.
Docs, CI's not-built list, NOTICE and install_dependencies.bash follow.

Tested: cho_task_manager 578, cho_robot_config 203, cho_bringup_common 313,
cho_description_franka 30, cho_bringup_franka 24, cho_simulation_isaac 14,
launch goldens 121 pass; headers pass. MuJoCo controller_check_torque on the
default robot (xml/fr3) and on the project's FT robot through its wrapper:
every torque controller and the gripper, SUCCESS. Isaac and the real robot
not run.

File: cho_description/cho_description_franka/robots/common/franka_robot.xacro (robot description, xacro)
@@ -19,4 +19,5 @@
                       ee_id:=none
                       special_connection:=''
+                      ee_connection_xacro:=''
                       gazebo:='false'
                       with_sc:='false'
@@ -49,72 +50,11 @@
       connected_to="${connected_to}"
     />
-    <!-- Bota SensONE Force-Torque Sensor -->
-    <xacro:unless value="${special_connection == ''}">
-      <!-- Mounting part bolted to the arm flange (link8) -->
-      <joint name="robot_mounting_link_to_bota_ft_sensor" type="fixed">
-        <parent link="${arm_prefix}${robot_type}_link8"/>
-        <child link="bota_ft_sensor_mounting"/>
-        <origin rpy="0 0 0" xyz="0 0 0"/>
-      </joint>
-      <link name="bota_ft_sensor_mounting">
-        <inertial>
-          <origin rpy="0 0 0" xyz="-0.00011559 0.00060052 0.010067"/>
-          <mass value="0.15393"/>
-          <inertia ixx="4.907E-05" ixy="3.2541E-08" ixz="-1.0415E-07" iyy="5.5735E-05" iyz="1.3709E-07" izz="9.0228E-05"/>
-        </inertial>
-        <visual>
-          <origin rpy="0 0 0" xyz="0 0 0"/>
-          <geometry>
-            <mesh filename="package://cho_description_franka/meshes/accessories/ft_sensor/mounting.stl"/>
-          </geometry>
-          <material name="bota_ft_material">
-            <color rgba="0.6902 0.61176 0.52941 1"/>
-          </material>
-        </visual>
-        <collision>
-          <origin rpy="0 0 0" xyz="0 0 0.011"/>
-          <geometry><cylinder length="0.028" radius="0.035"/></geometry>
-        </collision>
-        <collision>
-          <origin rpy="1.57 0 0" xyz="0 0.051 0.0115"/>
-          <geometry><cylinder length="0.032" radius="0.0065"/></geometry>
-        </collision>
-        <collision>
-          <origin rpy="0 0 0" xyz="0 0 0.03"/>
-          <geometry><cylinder length="0.01" radius="0.0315"/></geometry>
-        </collision>
-      </link>
-      <!-- Wrench (force/torque measurement) frame, 35 mm above the mounting base -->
-      <joint name="bota_ft_sensor_mounting_to_wrench" type="fixed">
-        <origin rpy="0 0 0" xyz="0 0 0.035"/>
-        <parent link="bota_ft_sensor_mounting"/>
-        <child link="bota_ft_sensor_wrench"/>
-      </joint>
-      <link name="bota_ft_sensor_wrench">
-        <inertial>
-          <origin rpy="0 0 0" xyz="-0.00018335 -3.3341E-07 -0.0070612"/>
-          <mass value="0.08253"/>
-          <inertia ixx="2.2674E-05" ixy="-3.9222E-12" ixz="4.8952E-08" iyy="2.2294E-05" iyz="4.0972E-11" izz="4.0919E-05"/>
-        </inertial>
-      </link>
-      <!-- Internal mechanical reference frames -->
-      <joint name="bota_ft_sensor_mounting_to_mech1" type="fixed">
-        <origin rpy="1.5625 0 -1.5708" xyz="-0.032879 0 0.0105"/>
-        <parent link="bota_ft_sensor_mounting"/>
-        <child link="bota_ft_sensor_mech1"/>
-      </joint>
-      <link name="bota_ft_sensor_mech1"/>
-      <joint name="bota_ft_sensor_mounting_to_mech2" type="fixed">
-        <origin rpy="1.5708 0 0" xyz="0 -0.032879 0.0105"/>
-        <parent link="bota_ft_sensor_mounting"/>
-        <child link="bota_ft_sensor_mech2"/>
-      </joint>
-      <link name="bota_ft_sensor_mech2"/>
-      <joint name="bota_ft_sensor_mounting_to_mech3" type="fixed">
-        <origin rpy="1.5708 0 1.5708" xyz="0.032879 0 0.0105"/>
-        <parent link="bota_ft_sensor_mounting"/>
-        <child link="bota_ft_sensor_mech3"/>
-      </joint>
-      <link name="bota_ft_sensor_mech3"/>
+    <!-- What a project mounts between the flange (link8) and the end effector, a
+         force-torque sensor for one: ee_connection_xacro names a xacro file whose
+         ee_connection(arm_prefix, robot_type) macro adds those links from link8, and
+         special_connection the link the end effector then hangs off. -->
+    <xacro:unless value="${ee_connection_xacro == ''}">
+      <xacro:include filename="${ee_connection_xacro}"/>
+      <xacro:ee_connection arm_prefix="${arm_prefix}" robot_type="${robot_type}"/>
     </xacro:unless>
     <xacro:if value="${hand and ee_id == 'franka_hand'}">
@@ -127,5 +67,5 @@
         <xacro:property name="ee_color" value="white" />
       </xacro:if>
-      <xacro:property name="connection" value="${'bota_ft_sensor_wrench' if special_connection != '' else robot_type + '_link8'}" />
+      <xacro:property name="connection" value="${special_connection if special_connection != '' else robot_type + '_link8'}" />
       <xacro:franka_hand
         connected_to="${arm_prefix}${connection}"
@@ -147,5 +87,5 @@
       <xacro:include filename="$(find cho_description_franka)/end_effectors/common/ee_with_one_link.xacro"/>
       <xacro:include filename="$(find cho_description_franka)/end_effectors/common/utils.xacro" />
-      <xacro:property name="connection" value="${'bota_ft_sensor_wrench' if special_connection != '' else robot_type + '_link8'}" />
+      <xacro:property name="connection" value="${special_connection if special_connection != '' else robot_type + '_link8'}" />
       <xacro:ee_with_one_link
         connected_to="${arm_prefix}${connection}"

File: cho_description/cho_description_franka/robots/fr3/fr3.urdf.xacro (robot description, xacro)
@@ -15,4 +15,7 @@
   <!-- Where is the end-effector connected to, if different from the robot flange?  -->
   <xacro:arg name="special_connection" default="" />
+  <!-- A xacro file whose ee_connection() macro mounts parts between the flange and that
+       link (robots/common/franka_robot.xacro); empty mounts nothing. -->
+  <xacro:arg name="ee_connection_xacro" default="" />
   <!-- Position offset between ee and parent frame -->
   <xacro:arg name="xyz_ee" default="0 0 0" />
@@ -56,4 +59,5 @@
                       ee_id="$(arg ee_id)"
                       special_connection="$(arg special_connection)"
+                      ee_connection_xacro="$(arg ee_connection_xacro)"
                       xyz_ee="$(arg xyz_ee)"
                       rpy_ee="$(arg rpy_ee)"
